Commit message: done add base

File: Open_arm_a1_ws/openarm_description/urdf/body/openarm_body.xacro (robot description, xacro)
@@ -11,9 +11,12 @@
                        inertials:=''
                        kinematics:=''
-                       kinematics_link:=''">
+                       kinematics_link:=''
+                       create_connected_link:=true">
     <xacro:property name="prefix" value="${'' if no_prefix else 'openarm_body_'}" />
     <!-- Connect the body to the world -->
     <xacro:if value="${connected_to != ''}">
-      <link name="${connected_to}" />
+      <xacro:if value="${create_connected_link}">
+        <link name="${connected_to}" />
+      </xacro:if>
       <joint name="${prefix}joint_to_${connected_to}" type="fixed">
         <parent link="${connected_to}" />

File: Open_arm_a1_ws/openarm_description/urdf/robot/openarm_robot.xacro (robot description, xacro)
@@ -38,8 +38,16 @@
             right_arm_prefix:='right_'
             can_fd:='true'
+            mobile_base:=false
+            mobile_base_xyz:='0 0 0'
+            mobile_base_rpy:='0 0 0'
+            mobile_base_arm_xyz:='0 0 0'
+            mobile_base_arm_rpy:='0 0 0'
+            mobile_base_body_xyz:='0 0 0'
+            mobile_base_body_rpy:='0 0 0'
             "
             >
     <xacro:include filename="$(find openarm_description)/urdf/arm/openarm_macro.xacro" />
     <xacro:include filename="$(find openarm_description)/urdf/arm/openarm_arm.xacro" />
+    <xacro:include filename="$(find openarm_description)/urdf/base/openarm_base.xacro" />
     <xacro:include filename="$(find openarm_description)/urdf/body/openarm_body_macro.xacro" />
     <xacro:include filename="$(find openarm_description)/urdf/body/openarm_body.xacro" />
@@ -53,4 +61,12 @@
     <xacro:property name="arm_prefix_modified" value="${'' if arm_prefix == '' else arm_prefix + '_'}" />
     <xacro:property name="body_prefix_modified" value="${'' if body_prefix == '' else body_prefix + '_'}" />
+    <xacro:property name="base_link_name" value="openarm_base_link" />
+    <xacro:if value="${mobile_base}">
+        <xacro:openarm_base
+        description_pkg="openarm_description"
+        connected_to="${body_connected_to}"
+        xyz="${mobile_base_xyz}"
+        rpy="${mobile_base_rpy}" />
+    </xacro:if>
     <xacro:if value="${bimanual}">
         <xacro:openarm_body
@@ -59,10 +75,11 @@
         no_prefix="${no_prefix}"
         description_pkg="openarm_description"
-        connected_to="${body_connected_to}"
-        xyz="${xyz}"
-        rpy="${rpy}"
+        connected_to="${base_link_name if mobile_base else body_connected_to}"
+        xyz="${mobile_base_body_xyz if mobile_base else xyz}"
+        rpy="${mobile_base_body_rpy if mobile_base else rpy}"
         inertials="${body_inertials}"
         kinematics="${body_kinematics}"
-        kinematics_link="${body_kinematics_link}" />
+        kinematics_link="${body_kinematics_link}"
+        create_connected_link="${not mobile_base}" />
         <!-- left arm -->
         <xacro:openarm_arm
@@ -140,11 +157,11 @@
         arm_prefix="${arm_prefix_modified}"
         no_prefix="${no_prefix}"
-        xyz="${xyz}"
-        rpy="${rpy}"
+        xyz="${mobile_base_arm_xyz if mobile_base else xyz}"
+        rpy="${mobile_base_arm_rpy if mobile_base else rpy}"
         joint_limits="${joint_limits}"
         kinematics="${kinematics}"
         kinematics_link="${kinematics_link}"
         inertials="${inertials}"
-        connected_to=""
+        connected_to="${base_link_name if mobile_base else ''}"
         />
         <xacro:if value="${ros2_control}">

File: Open_arm_a1_ws/openarm_description/urdf/robot/v10.urdf.xacro (robot description, xacro)
@@ -27,4 +27,11 @@
   <xacro:arg name="left_arm_base_rpy" default="-1.5708 0 0" />
   <xacro:arg name="can_fd" default="true" />
+  <xacro:arg name="mobile_base" default="false" />
+  <xacro:arg name="mobile_base_xyz" default="0 0 0" />
+  <xacro:arg name="mobile_base_rpy" default="0 0 0" />
+  <xacro:arg name="mobile_base_arm_xyz" default="0 0 0" />
+  <xacro:arg name="mobile_base_arm_rpy" default="0 0 0" />
+  <xacro:arg name="mobile_base_body_xyz" default="0 0 0" />
+  <xacro:arg name="mobile_base_body_rpy" default="0 0 0" />
   <xacro:openarm_robot
   arm_type="v10"
@@ -61,4 +68,11 @@
   left_arm_base_rpy="$(arg left_arm_base_rpy)"
   can_fd="$(arg can_fd)"
+  mobile_base="$(arg mobile_base)"
+  mobile_base_xyz="$(arg mobile_base_xyz)"
+  mobile_base_rpy="$(arg mobile_base_rpy)"
+  mobile_base_arm_xyz="$(arg mobile_base_arm_xyz)"
+  mobile_base_arm_rpy="$(arg mobile_base_arm_rpy)"
+  mobile_base_body_xyz="$(arg mobile_base_body_xyz)"
+  mobile_base_body_rpy="$(arg mobile_base_body_rpy)"
   />
 </robot>
