Commit message: feat: integrate body v1 components with updated URDF parameters and mesh assets

File: Open_arm_a1_ws/src/openarm_description/urdf/body/openarm_body.xacro (robot description, xacro)
@@ -25,35 +25,23 @@
       </joint>
     </xacro:if>
-    <!-- ========================================================================= -->
-    <!-- CHANGING THE BODY                                                         -->
-    <!-- ========================================================================= -->
-    <!-- If you design a new body (like an AGV, a new stand, etc.):                -->
-    <!-- 1. Drop the new meshes into meshes/body/v10/visual/ and collision/        -->
-    <!-- 2. Change the filename="..." below to match your new mesh names.          -->
-    <!-- 3. Update the mass and inertia directly in the <inertial> tag below.      -->
-    <!-- 4. Need wheels or extra links? Just add new <link> and <joint> tags here! -->
-    <!-- ========================================================================= -->
     <link name="${prefix}link0">
       <visual>
-        <origin xyz="0 0 0" rpy="0 0 0" />
+        <origin xyz="-0.251 0.1302 -0.210104" rpy="0 0 -1.5708" />
         <geometry>
-          <!-- Swap the visual mesh here -->
-          <mesh filename="package://${description_pkg}/meshes/body/${body_type}/visual/body_link0.dae" scale="0.001 0.001 0.001" />
+          <mesh filename="package://${description_pkg}/meshes/body/${body_type}/visual/body_link0.STL" scale="0.001 0.001 0.001" />
         </geometry>
       </visual>
       <collision>
-        <origin xyz="0 0 0" rpy="0 0 0" />
+        <origin xyz="-0.251 0.1302 -0.210104" rpy="0 0 -1.5708" />
         <geometry>
-          <!-- Swap the collision mesh here -->
-          <mesh filename="package://${description_pkg}/meshes/body/${body_type}/collision/body_link0_symp.stl" scale="0.001 0.001 0.001" />
+          <mesh filename="package://${description_pkg}/meshes/body/${body_type}/collision/body_link0_symp.STL" scale="0.001 0.001 0.001" />
         </geometry>
       </collision>
-      <!-- Mass and Inertia (from configuration/common_version/tomo_alpha style) -->
       <inertial>
-        <origin xyz="0 0 0" rpy="0 0 0" />
-        <mass value="13.89" />
-        <inertia ixx="1.653" ixy="0.0" ixz="0.0"
-                 iyy="1.653" iyz="0.0"
-                 izz="0.051" />
+        <origin xyz="-0.026141 4.0416E-06 0.40173" rpy="0 0 0" />
+        <mass value="3.0436" />
+        <inertia ixx="0.14438" ixy="1.054E-06" ixz="1.0507E-06"
+                 iyy="0.14207" iyz="9.0865E-10"
+                 izz="0.019727" />
       </inertial>
     </link>

File: Open_arm_a1_ws/src/openarm_description/urdf/robot/v10.urdf.xacro (robot description, xacro)
@@ -3,5 +3,5 @@
   <xacro:include filename="$(find openarm_description)/urdf/robot/openarm_robot.xacro"/>
   <xacro:arg name="arm_type" default="v10" />
-  <xacro:arg name="body_type" default="v10" />
+  <xacro:arg name="body_type" default="v1" />
   <xacro:arg name="ee_type" default="openarm_hand" />
   <xacro:arg name="no_prefix" default="false"/>
@@ -22,7 +22,7 @@
   <xacro:arg name="fake_sensor_commands" default="false" />
   <xacro:arg name="bimanual" default="false" />
-  <xacro:arg name="right_arm_base_xyz" default="0.0 -0.031 0.698" />
+  <xacro:arg name="right_arm_base_xyz" default="-0.0964262 -0.1302 0.836" />
   <xacro:arg name="right_arm_base_rpy" default="1.5708 0 0" />
-  <xacro:arg name="left_arm_base_xyz" default="0.0 0.031 0.698" />
+  <xacro:arg name="left_arm_base_xyz" default="-0.0964262 0.1302 0.836" />
   <xacro:arg name="left_arm_base_rpy" default="-1.5708 0 0" />
   <xacro:arg name="can_fd" default="true" />
@@ -33,8 +33,8 @@
   <xacro:arg name="mobile_base_arm_rpy" default="0 0 0" />
   <xacro:arg name="mobile_base_body_xyz" default="0 0 0" />
-  <xacro:arg name="mobile_base_body_rpy" default="0 0 0" />
+  <xacro:arg name="mobile_base_body_rpy" default="0 0 3.14159" />
   <xacro:openarm_robot
   arm_type="v10"
-  body_type="v10"
+  body_type="v1"
   joint_limits="${xacro.load_yaml('$(find openarm_description)/config/arm/v10/joint_limits.yaml')}"
   control_gains="${xacro.load_yaml('$(find openarm_description)/config/arm/v10/control_gains.yaml')}"
@@ -43,7 +43,7 @@
   kinematics_link="${xacro.load_yaml('$(find openarm_description)/config/arm/v10/kinematics_link.yaml')}"
   kinematics_offset="${xacro.load_yaml('$(find openarm_description)/config/arm/v10/kinematics_offset.yaml')}"
-  body_inertials="${xacro.load_yaml('$(find openarm_description)/config/body/v10/inertials.yaml')}"
-  body_kinematics="${xacro.load_yaml('$(find openarm_description)/config/body/v10/kinematics.yaml')}"
-  body_kinematics_link="${xacro.load_yaml('$(find openarm_description)/config/body/v10/kinematics.yaml')}"
+  body_inertials="${xacro.load_yaml('$(find openarm_description)/config/body/v1/inertials.yaml')}"
+  body_kinematics="${xacro.load_yaml('$(find openarm_description)/config/body/v1/kinematics.yaml')}"
+  body_kinematics_link="${xacro.load_yaml('$(find openarm_description)/config/body/v1/kinematics_link.yaml')}"
   ee_kinematics_link="${xacro.load_yaml('$(find openarm_description)/config/hand/openarm_hand/kinematics_link.yaml')}"
   hand="$(arg hand)"
