Commit message: Update URDF and XACRO files for amazing hand model
- Added collision geometries for distal and proximal links in r_ahand.urdf and r_ahand_macro.xacro to enhance physical interactions.
- Changed joint definitions from 'joint' to 'mimic' for several joints in both r_ahand.urdf and r_ahand_macro.xacro to improve control behavior.
- Updated body type argument from 'v1' to 'v2' in v10.urdf.xacro to reflect the latest design specifications.

File: Open_arm_a1_ws/src/openarm_description/urdf/body/openarm_body.xacro (robot description, xacro)
@@ -25,25 +25,103 @@
       </joint>
     </xacro:if>
+    <!-- v2's chassis mesh (chasssis_link.STL, base-plate component stripped out) is
+         already centered on its mount point, already in meters, and carries its own
+         correctly-measured inertial; v1/v10's raw mesh is in mm and isn't centered,
+         so they need the baked-in offset + scale instead. -->
+    <xacro:property name="mesh_xyz" value="${'0 0 0' if body_type == 'v2' else '-0.251 0.1302 -0.210104'}" />
+    <xacro:property name="mesh_rpy" value="${'0 0 0' if body_type == 'v2' else '0 0 -1.5708'}" />
+    <xacro:property name="mesh_scale" value="${'1 1 1' if body_type == 'v2' else '0.001 0.001 0.001'}" />
     <link name="${prefix}link0">
       <visual>
-        <origin xyz="-0.251 0.1302 -0.210104" rpy="0 0 -1.5708" />
+        <origin xyz="${mesh_xyz}" rpy="${mesh_rpy}" />
         <geometry>
-          <mesh filename="package://${description_pkg}/meshes/body/${body_type}/visual/body_link0.STL" scale="0.001 0.001 0.001" />
+          <mesh filename="package://${description_pkg}/meshes/body/${body_type}/visual/body_link0.STL" scale="${mesh_scale}" />
         </geometry>
       </visual>
       <collision>
-        <origin xyz="-0.251 0.1302 -0.210104" rpy="0 0 -1.5708" />
+        <origin xyz="${mesh_xyz}" rpy="${mesh_rpy}" />
         <geometry>
-          <mesh filename="package://${description_pkg}/meshes/body/${body_type}/collision/body_link0_symp.STL" scale="0.001 0.001 0.001" />
+          <mesh filename="package://${description_pkg}/meshes/body/${body_type}/collision/body_link0_symp.STL" scale="${mesh_scale}" />
         </geometry>
       </collision>
-      <inertial>
-        <origin xyz="-0.026141 4.0416E-06 0.40173" rpy="0 0 0" />
-        <mass value="3.0436" />
-        <inertia ixx="0.14438" ixy="1.054E-06" ixz="1.0507E-06"
-                 iyy="0.14207" iyz="9.0865E-10"
-                 izz="0.019727" />
-      </inertial>
+      <xacro:unless value="${body_type == 'v2'}">
+        <inertial>
+          <origin xyz="-0.026141 4.0416E-06 0.40173" rpy="0 0 0" />
+          <mass value="3.0436" />
+          <inertia ixx="0.14438" ixy="1.054E-06" ixz="1.0507E-06"
+                   iyy="0.14207" iyz="9.0865E-10"
+                   izz="0.019727" />
+        </inertial>
+      </xacro:unless>
+      <xacro:if value="${body_type == 'v2'}">
+        <inertial>
+          <origin xyz="-0.050424 -0.0013901 -0.23707" rpy="0 0 0" />
+          <mass value="25" />
+          <inertia ixx="0.053286" ixy="0.00012916" ixz="2.3176E-06"
+                   iyy="0.044721" iyz="0.00046953"
+                   izz="0.047419" />
+        </inertial>
+      </xacro:if>
     </link>
+    <!-- v2 adds an articulated neck + head; older body versions are a single rigid
+         chassis with no such thing, so this is entirely gated on body_type. -->
+    <xacro:if value="${body_type == 'v2'}">
+      <link name="${prefix}neck_link">
+        <visual>
+          <origin xyz="0 0 0" rpy="0 0 0" />
+          <geometry>
+            <mesh filename="package://${description_pkg}/meshes/body/${body_type}/visual/Neck_Link.STL" />
+          </geometry>
+        </visual>
+        <collision>
+          <origin xyz="0 0 0" rpy="0 0 0" />
+          <geometry>
+            <mesh filename="package://${description_pkg}/meshes/body/${body_type}/collision/Neck_Link_symp.STL" />
+          </geometry>
+        </collision>
+        <inertial>
+          <origin xyz="-0.00729797698843204 -0.000443616169626848 -0.0174999999999999" rpy="0 0 0" />
+          <mass value="0.0279371439221494" />
+          <inertia ixx="6.39092695773795E-06" ixy="-5.69576500715137E-09" ixz="-1.75825511004272E-20"
+                   iyy="6.48428237240793E-06" iyz="2.37840275503138E-21"
+                   izz="7.48673899437131E-06" />
+        </inertial>
+      </link>
+      <joint name="${prefix}neck_joint" type="revolute">
+        <origin xyz="-0.031878 0.023312 0.33482" rpy="-1.8793 1.5431 -0.30844" />
+        <parent link="${prefix}link0" />
+        <child link="${prefix}neck_link" />
+        <axis xyz="0 0 -1" />
+        <limit lower="-1.57" upper="1.57" effort="10" velocity="3" />
+      </joint>
+      <link name="${prefix}head_link">
+        <visual>
+          <origin xyz="0 0 0" rpy="0 0 0" />
+          <geometry>
+            <mesh filename="package://${description_pkg}/meshes/body/${body_type}/visual/Head_Link.STL" />
+          </geometry>
+        </visual>
+        <collision>
+          <origin xyz="0 0 0" rpy="0 0 0" />
+          <geometry>
+            <mesh filename="package://${description_pkg}/meshes/body/${body_type}/collision/Head_Link_symp.STL" />
+          </geometry>
+        </collision>
+        <inertial>
+          <origin xyz="0.0353707921732529 -0.00624420290577887 0.140058128714488" rpy="0 0 0" />
+          <mass value="2.4504028411393" />
+          <inertia ixx="0.0238556395901539" ixy="-0.000356410646591372" ixz="0.00130415554911385"
+                   iyy="0.0179669744913406" iyz="8.15599537572202E-05"
+                   izz="0.0155300891818827" />
+        </inertial>
+      </link>
+      <joint name="${prefix}head_joint" type="revolute">
+        <origin xyz="-0.023265 0.00306 -0.01733" rpy="1.5364 0 -1.5444" />
+        <parent link="${prefix}neck_link" />
+        <child link="${prefix}head_link" />
+        <axis xyz="0.034355 -0.034358 0.99882" />
+        <limit lower="-1.57" upper="1.57" effort="10" velocity="3" />
+      </joint>
+    </xacro:if>
   </xacro:macro>
 </robot>

File: Open_arm_a1_ws/src/openarm_description/urdf/ee/amazing_hand/l_ahand.urdf (robot description, URDF)
Before this commit: robot left_hand, 123 links, 122 joints
Links:
- link distal: geometry collision cylinder length=0.042048 radius=0.0136333; visual mesh filename=package://openarm_description/meshes/ee/amazing_hand/left/D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 scale=1 1 1
- link distal_1: geometry collision cylinder length=0.042048 radius=0.0136333; visual mesh filename=package://openarm_description/meshes/ee/amazing_hand/left/D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 scale=1 1 1
- link distal_2: geometry collision cylinder length=0.042048 radius=0.0136333; visual mesh filename=package://openarm_description/meshes/ee/amazing_hand/left/D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 scale=1 1 1
- link distal_3: geometry collision cylinder length=0.042048 radius=0.0136333; visual mesh filename=package://openarm_description/meshes/ee/amazing_hand/left/D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 scale=1 1 1
- link proximal: geometry collision cylinder length=0.0239747 radius=0.0224239; visual mesh filename=package://openarm_description/meshes/ee/amazing_hand/left/P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 scale=1 1 1
- link proximal_1: geometry collision cylinder length=0.0239747 radius=0.0224239; visual mesh filename=package://openarm_description/meshes/ee/amazing_hand/left/P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 scale=1 1 1
- link proximal_2: geometry collision cylinder length=0.0239747 radius=0.0224239; visual mesh filename=package://openarm_description/meshes/ee/amazing_hand/left/P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 scale=1 1 1
- link proximal_3: geometry collision cylinder length=0.0239747 radius=0.0224239; visual mesh filename=package://openarm_description/meshes/ee/amazing_hand/left/P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 scale=1 1 1
Joints:
- joint cylindrical_1_1: mimic (none) -> joint=j21 multiplier=-0.856286 offset=-0.038898
- joint cylindrical_1_3: mimic (none) -> joint=j22 multiplier=-0.856286 offset=-0.038898
- joint cylindrical_1_5: mimic (none) -> joint=j23 multiplier=-0.856286 offset=-0.038898
- joint cylindrical_1_7: mimic (none) -> joint=j24 multiplier=-0.856286 offset=-0.038898
- joint revolute_1: mimic (none) -> joint=j11 multiplier=1 offset=0
- joint revolute_1_1: mimic (none) -> joint=j12 multiplier=1 offset=0
- joint revolute_1_2: mimic (none) -> joint=j13 multiplier=1 offset=0
- joint revolute_1_4: mimic (none) -> joint=j14 multiplier=1 offset=0
- joint revolute_2: mimic (none) -> joint=j21 multiplier=-1.0 offset=0
- joint revolute_2_1: mimic (none) -> joint=j22 multiplier=-1.0 offset=0
- joint revolute_2_2: mimic (none) -> joint=j23 multiplier=-1.0 offset=0
- joint revolute_2_3: mimic (none) -> joint=j24 multiplier=-1.0 offset=0
- joint revolute_3_1: mimic (none) -> joint=j21 multiplier=1.062201 offset=-0.015673
- joint revolute_3_2: mimic (none) -> joint=j22 multiplier=1.062201 offset=-0.015673
- joint revolute_3_3: mimic (none) -> joint=j23 multiplier=1.062201 offset=-0.015673
- joint revolute_3_4: mimic (none) -> joint=j24 multiplier=1.062201 offset=-0.015673
- joint revolute_5: mimic (none) -> joint=j21 multiplier=1.019021 offset=0.037525
- joint revolute_5_1: mimic (none) -> joint=j22 multiplier=1.019021 offset=0.037525
- joint revolute_5_2: mimic (none) -> joint=j23 multiplier=1.019021 offset=0.037525
- joint revolute_5_3: mimic (none) -> joint=j24 multiplier=1.019021 offset=0.037525
- joint revolute_6: mimic (none) -> joint=j21 multiplier=-1.019022 offset=-0.037525
- joint revolute_6_1: mimic (none) -> joint=j22 multiplier=-1.019022 offset=-0.037525
- joint revolute_6_2: mimic (none) -> joint=j23 multiplier=-1.019022 offset=-0.037525
- joint revolute_6_3: mimic (none) -> joint=j24 multiplier=-1.019022 offset=-0.037525

File: Open_arm_a1_ws/src/openarm_description/urdf/ee/amazing_hand/l_ahand_macro.xacro (robot description, xacro)
@@ -249,5 +249,5 @@
                 <color rgba="1 1 1 1" />
             </material>
-        </visual></link>
+        </visual><collision><origin xyz="0.001403314127 0.0233651278 -0.002288079611" rpy="3.141592654 -1.256637061 1.884955592" /><geometry><cylinder radius="0.0136333" length="0.042048" /></geometry></collision></link>
     <link name="${prefix}distal_1">
         <inertial>
@@ -272,5 +272,5 @@
                 <color rgba="1 1 1 1" />
             </material>
-        </visual></link>
+        </visual><collision><origin xyz="0.001403314127 0.0233651278 -0.002288079611" rpy="3.141592654 -1.256637061 1.884955592" /><geometry><cylinder radius="0.0136333" length="0.042048" /></geometry></collision></link>
     <link name="${prefix}distal_2">
         <inertial>
@@ -295,5 +295,5 @@
                 <color rgba="1 1 1 1" />
             </material>
-        </visual></link>
+        </visual><collision><origin xyz="0.001403314127 0.0233651278 -0.002288079611" rpy="-3.141592654 -1.256637061 1.884955592" /><geometry><cylinder radius="0.0136333" length="0.042048" /></geometry></collision></link>
     <link name="${prefix}distal_3">
         <inertial>
@@ -318,5 +318,5 @@
                 <color rgba="1 1 1 1" />
             </material>
-        </visual></link>
+        </visual><collision><origin xyz="0.001403314127 0.0233651278 -0.002288079611" rpy="3.141592654 -1.256637061 1.884955592" /><geometry><cylinder radius="0.0136333" length="0.042048" /></geometry></collision></link>
     <link name="${prefix}distal__1__loop_closure">
         <inertial>
@@ -593,5 +593,5 @@
                 <color rgba="1 1 1 1" />
             </material>
-        </visual></link>
+        </visual><collision><origin xyz="0.007113500402 0.03005137885 0.008107388089" rpy="-0.1291687974 -1.254170147 0.1228140104" /><geometry><cylinder radius="0.0224239" length="0.0239747" /></geometry></collision></link>
     <link name="${prefix}proximal_1">
         <inertial>
@@ -616,5 +616,5 @@
                 <color rgba="1 1 1 1" />
             </material>
-        </visual></link>
+        </visual><collision><origin xyz="0.007113500402 0.03005137885 0.008107388089" rpy="-0.1291687974 -1.254170147 0.1228140104" /><geometry><cylinder radius="0.0224239" length="0.0239747" /></geometry></collision></link>
     <link name="${prefix}proximal_2">
         <inertial>
@@ -639,5 +639,5 @@
                 <color rgba="1 1 1 1" />
             </material>
-        </visual></link>
+        </visual><collision><origin xyz="0.007113500402 0.03005137885 0.008107388089" rpy="-0.1291687974 -1.254170147 0.1228140104" /><geometry><cylinder radius="0.0224239" length="0.0239747" /></geometry></collision></link>
     <link name="${prefix}proximal_3">
         <inertial>
@@ -662,5 +662,5 @@
                 <color rgba="1 1 1 1" />
             </material>
-        </visual></link>
+        </visual><collision><origin xyz="0.007113500402 0.03005137885 0.008107388089" rpy="-0.1291687974 -1.254170147 0.1228140104" /><geometry><cylinder radius="0.0224239" length="0.0239747" /></geometry></collision></link>
     <link name="${prefix}l_hand_plate">
         <inertial>
@@ -1390,5 +1390,5 @@
         <parent link="${prefix}cylindrical_1" />
         <child link="${prefix}distal_2" />
-    </joint>
+    <mimic joint="${prefix[:-6]}j21" multiplier="-0.856286" offset="-0.038898" /></joint>
     <joint name="${prefix}cylindrical_1_2" type="prismatic">
         <origin xyz="-0.00035 0.0496106 0.00943613" rpy="-0.0804909 5.31725e-17 -1.07388e-15" />
@@ -1403,5 +1403,5 @@
         <parent link="${prefix}cylindrical_1_1" />
         <child link="${prefix}distal_1" />
-    </joint>
+    <mimic joint="${prefix[:-6]}j22" multiplier="-0.856286" offset="-0.038898" /></joint>
     <joint name="${prefix}cylindrical_1_4" type="prismatic">
         <origin xyz="-0.00035 0.0496106 0.00943613" rpy="-0.0804909 1.6886e-15 -1.81943e-15" />
@@ -1416,5 +1416,5 @@
         <parent link="${prefix}cylindrical_1_2" />
         <child link="${prefix}distal_3" />
-    </joint>
+    <mimic joint="${prefix[:-6]}j23" multiplier="-0.856286" offset="-0.038898" /></joint>
     <joint name="${prefix}cylindrical_1_6" type="prismatic">
         <origin xyz="-0.00035 0.0496106 0.00943613" rpy="-0.0804909 -5.59989e-17 -5.25791e-16" />
@@ -1429,5 +1429,5 @@
         <parent link="${prefix}cylindrical_1_3" />
         <child link="${prefix}distal" />
-    </joint>
+    <mimic joint="${prefix[:-6]}j24" multiplier="-0.856286" offset="-0.038898" /></joint>
     <joint name="${prefix}fastened_1" type="fixed">
         <origin xyz="0.00605 -0.01245 -0.008" rpy="1.5708 -1.12906e-14 3.14159" />
@@ -1664,5 +1664,5 @@
         <child link="${prefix}gimbal_2" />
         <limit effort="1" velocity="1" lower="-0.349066" upper="0.349066" />
-    </joint>
+    <mimic joint="${prefix[:-6]}j11" multiplier="1" offset="0" /></joint>
     <joint name="${prefix}revolute_1_1" type="revolute">
         <origin xyz="-6.93889e-18 -6.93889e-18 0.001" rpy="-3.14159 2.05193e-27 4.1595e-14" />
@@ -1671,5 +1671,5 @@
         <child link="${prefix}gimbal_1" />
         <limit effort="1" velocity="1" lower="-0.349066" upper="0.349066" />
-    </joint>
+    <mimic joint="${prefix[:-6]}j12" multiplier="1" offset="0" /></joint>
     <joint name="${prefix}revolute_1_2" type="revolute">
         <origin xyz="-9.02056e-17 -4.85723e-17 0.001" rpy="3.14159 -2.01489e-16 -6.93889e-16" />
@@ -1678,5 +1678,5 @@
         <child link="${prefix}gimbal_3" />
         <limit effort="1" velocity="1" lower="-0.349066" upper="0.349066" />
-    </joint>
+    <mimic joint="${prefix[:-6]}j13" multiplier="1" offset="0" /></joint>
     <joint name="${prefix}revolute_1_3" type="continuous">
         <origin xyz="-0.00526725 0.0291633 -0.003" rpy="1.6093e-16 -1.30023e-16 0.10472" />
@@ -1691,5 +1691,5 @@
         <child link="${prefix}gimbal" />
         <limit effort="1" velocity="1" lower="-0.349066" upper="0.349066" />
-    </joint>
+    <mimic joint="${prefix[:-6]}j14" multiplier="1" offset="0" /></joint>
     <joint name="${prefix}revolute_2" type="revolute">
         <origin xyz="-0.00525 -1.73472e-17 -0.0035" rpy="-1.80303e-13 -9.84526e-17 1.69309e-15" />
@@ -1698,5 +1698,5 @@
         <child link="${prefix}proximal_2" />
         <limit effort="1" velocity="1" lower="-1.35615" upper="0.0924772" />
-    </joint>
+    <mimic joint="${prefix[:-6]}j21" multiplier="-1.0" offset="0" /></joint>
     <joint name="${prefix}revolute_2_1" type="revolute">
         <origin xyz="-0.00525 6.93889e-18 -0.0035" rpy="-1.60745e-14 -4.74371e-17 5.18347e-15" />
@@ -1705,5 +1705,5 @@
         <child link="${prefix}proximal_1" />
         <limit effort="1" velocity="1" lower="-1.35615" upper="0.0924772" />
-    </joint>
+    <mimic joint="${prefix[:-6]}j22" multiplier="-1.0" offset="0" /></joint>
     <joint name="${prefix}revolute_2_2" type="revolute">
         <origin xyz="-0.00525 -9.02056e-17 -0.0035" rpy="-1.69048e-13 2.00624e-17 3.60822e-16" />
@@ -1712,5 +1712,5 @@
         <child link="${prefix}proximal_3" />
         <limit effort="1" velocity="1" lower="-1.35615" upper="0.0924772" />
-    </joint>
+    <mimic joint="${prefix[:-6]}j23" multiplier="-1.0" offset="0" /></joint>
     <joint name="${prefix}revolute_2_3" type="revolute">
         <origin xyz="-0.00525 -2.08167e-17 -0.0035" rpy="-4.9683e-16 7.86453e-17 1.45717e-16" />
@@ -1719,5 +1719,5 @@
         <child link="${prefix}proximal" />
         <limit effort="1" velocity="1" lower="-1.35615" upper="0.0924772" />
-    </joint>
+    <mimic joint="${prefix[:-6]}j24" multiplier="-1.0" offset="0" /></joint>
     <joint name="${prefix}revolute_2_4" type="continuous">
         <origin xyz="-0.00061573 -0.0150929 -0.003" rpy="-4.54497e-16 -6.24238e-16 1.5708" />
@@ -1737,5 +1737,5 @@
         <parent link="${prefix}gimbal_2" />
         <child link="${prefix}link_2" />
-    </joint>
+    <mimic joint="${prefix[:-6]}j21" multiplier="1.062201" offset="-0.015673" /></joint>
     <joint name="${prefix}revolute_3_2" type="continuous">
         <origin xyz="-0.0019 0 -0.0095" rpy="-9.90587e-15 -6.09448e-17 3.97123e-16" />
@@ -1743,5 +1743,5 @@
         <parent link="${prefix}gimbal_1" />
         <child link="${prefix}link_1" />
-    </joint>
+    <mimic joint="${prefix[:-6]}j22" multiplier="1.062201" offset="-0.015673" /></joint>
     <joint name="${prefix}revolute_3_3" type="continuous">
         <origin xyz="-0.0019 -5.55112e-17 -0.0095" rpy="-1.60716e-13 1.15478e-16 -3.33067e-16" />
@@ -1749,5 +1749,5 @@
         <parent link="${prefix}gimbal_3" />
         <child link="${prefix}link_3" />
-    </joint>
+    <mimic joint="${prefix[:-6]}j23" multiplier="1.062201" offset="-0.015673" /></joint>
     <joint name="${prefix}revolute_3_4" type="continuous">
         <origin xyz="-0.0019 -9.36751e-17 -0.0095" rpy="6.07431e-16 -9.9073e-16 2.56045e-15" />
@@ -1755,5 +1755,5 @@
         <parent link="${prefix}gimbal" />
         <child link="${prefix}link" />
-    </joint>
+    <mimic joint="${prefix[:-6]}j24" multiplier="1.062201" offset="-0.015673" /></joint>
     <joint name="${prefix}revolute_4" type="continuous">
         <origin xyz="-0.0270789 -0.0251197 -0.003" rpy="1.44071e-15 1.72452e-16 -3.3285e-16" />
@@ -1792,5 +1792,5 @@
         <child link="${prefix}custom_servo_horn_5" />
         <limit effort="1" velocity="1" lower="-2.18166" upper="0.959931" />
-    </joint>
+    <mimic joint="${prefix[:-6]}j21" multiplier="1.019021" offset="0.037525" /></joint>
     <joint name="${prefix}revolute_5_1" type="revolute">
         <origin xyz="-6.93889e-18 -0.0087 -0.01995" rpy="1.5708 -1.55931e-13 -2.47818e-16" />
@@ -1799,5 +1799,5 @@
         <child link="${prefix}custom_servo_horn_2" />
         <limit effort="1" velocity="1" lower="-2.18166" upper="0.959931" />
-    </joint>
+    <mimic joint="${prefix[:-6]}j22" multiplier="1.019021" offset="0.037525" /></joint>
     <joint name="${prefix}revolute_5_2" type="revolute">
         <origin xyz="-8.67362e-18 -0.0087 -0.01995" rpy="1.5708 8.76862e-15 -1.40489e-14" />
@@ -1806,5 +1806,5 @@
         <child link="${prefix}custom_servo_horn_6" />
         <limit effort="1" velocity="1" lower="-2.18166" upper="0.959931" />
-    </joint>
+    <mimic joint="${prefix[:-6]}j23" multiplier="1.019021" offset="0.037525" /></joint>
     <joint name="${prefix}revolute_5_3" type="revolute">
         <origin xyz="-1.04083e-17 -0.0087 -0.01995" rpy="1.5708 -1.96996e-15 -1.36945e-14" />
@@ -1813,5 +1813,5 @@
         <child link="${prefix}custom_servo_horn" />
         <limit effort="1" velocity="1" lower="-2.18166" upper="0.959931" />
-    </joint>
+    <mimic joint="${prefix[:-6]}j24" multiplier="1.019021" offset="0.037525" /></joint>
     <joint name="${prefix}revolute_6" type="revolute">
         <origin xyz="-2.08167e-17 -0.0087 -0.01995" rpy="-1.5708 1.54195e-15 3.14159" />
@@ -1820,5 +1820,5 @@
         <child link="${prefix}custom_servo_horn_4" />
         <limit effort="1" velocity="1" lower="-0.959931" upper="2.18166" />
-    </joint>
+    <mimic joint="${prefix[:-6]}j21" multiplier="-1.019022" offset="-0.037525" /></joint>
     <joint name="${prefix}revolute_6_1" type="revolute">
         <origin xyz="-2.77556e-17 -0.0087 -0.01995" rpy="-1.5708 2.88658e-15 3.14159" />
@@ -1827,5 +1827,5 @@
         <child link="${prefix}custom_servo_horn_3" />
         <limit effort="1" velocity="1" lower="-0.959931" upper="2.18166" />
-    </joint>
+    <mimic joint="${prefix[:-6]}j22" multiplier="-1.019022" offset="-0.037525" /></joint>
     <joint name="${prefix}revolute_6_2" type="revolute">
         <origin xyz="-1.34441e-17 -0.0087 -0.01995" rpy="-1.5708 -2.06903e-17 3.14159" />
@@ -1834,5 +1834,5 @@
         <child link="${prefix}custom_servo_horn_7" />
         <limit effort="1" velocity="1" lower="-0.959931" upper="2.18166" />
-    </joint>
+    <mimic joint="${prefix[:-6]}j23" multiplier="-1.019022" offset="-0.037525" /></joint>
     <joint name="${prefix}revolute_6_3" type="revolute">
         <origin xyz="-1.30104e-18 -0.0087 -0.01995" rpy="-1.5708 4.36477e-15 -3.14159" />
@@ -1841,5 +1841,5 @@
         <child link="${prefix}custom_servo_horn_1" />
         <limit effort="1" velocity="1" lower="-0.959931" upper="2.18166" />
-    </joint>
+    <mimic joint="${prefix[:-6]}j24" multiplier="-1.019022" offset="-0.037525" /></joint>
   </xacro:macro>
 </robot>
