Commit message: Fix joint references and update arm base positions in URDF files
- Updated mimic joint references in left and right hand URDF and XACRO files to correct joint mappings.
- Adjusted the base position and orientation parameters for the right and left arms in the robot's main XACRO file to ensure proper alignment.

File: Open_arm_a1_ws/src/openarm_description/urdf/body/openarm_body.xacro (robot description, xacro)
@@ -14,4 +14,15 @@
                        create_connected_link:=true">
     <xacro:property name="prefix" value="${'' if no_prefix else 'openarm_body_'}" />
+    <!-- No material tag = RViz's red fallback for untextured meshes. Colors match
+         the reference chassis_robot_description.urdf. -->
+    <material name="${prefix}chassis_light">
+      <color rgba="0.79216 0.81961 0.92941 1" />
+    </material>
+    <material name="${prefix}head_white">
+      <color rgba="1 1 1 1" />
+    </material>
+    <material name="${prefix}shell_white">
+      <color rgba="0.95 0.95 0.95 1" />
+    </material>
     <!-- Connect the body to the world -->
     <xacro:if value="${connected_to != ''}">
@@ -32,10 +43,6 @@
     <xacro:property name="head_mesh_xyz" value="0 0 0" />
     <xacro:property name="head_mesh_rpy" value="0 0 0" />
-    <!-- Outer cosmetic shell cover (RobotShell.STL). Came as a loose file with no
-         URDF of its own, so there's no reference joint origin to copy like the
-         chassis/neck/head had - start at identity and nudge from here. Note it's
-         in millimeters unlike the other v2 meshes, hence the scale. -->
-    <xacro:property name="shell_mesh_xyz" value="0.12 0 -0.27" />
-    <xacro:property name="shell_mesh_rpy" value="0 0 -1.5707" />
+    <xacro:property name="shell_mesh_xyz" value="0.1943 -14.5 -1.04" />
+    <xacro:property name="shell_mesh_rpy" value="0 0 1.5707" />
     <xacro:property name="shell_mesh_scale" value="0.001 0.001 0.001" />
     <link name="${prefix}link0">
@@ -45,4 +52,5 @@
           <mesh filename="package://${description_pkg}/meshes/body/${body_type}/visual/body_link0.STL" scale="${mesh_scale}" />
         </geometry>
+        <material name="${prefix}chassis_light" />
       </visual>
       <collision>
@@ -80,4 +88,5 @@
             <mesh filename="package://${description_pkg}/meshes/body/${body_type}/visual/Neck_Link.STL" />
           </geometry>
+          <material name="${prefix}chassis_light" />
         </visual>
         <collision>
@@ -108,4 +117,5 @@
             <mesh filename="package://${description_pkg}/meshes/body/${body_type}/visual/Head_Link.STL" />
           </geometry>
+          <material name="${prefix}head_white" />
         </visual>
         <collision>
@@ -138,4 +148,5 @@
             <mesh filename="package://${description_pkg}/meshes/body/${body_type}/visual/RobotShell.STL" scale="${shell_mesh_scale}" />
           </geometry>
+          <material name="${prefix}shell_white" />
         </visual>
       </link>

File: Open_arm_a1_ws/src/openarm_description/urdf/ee/amazing_hand/ahand.ros2_control.xacro (robot description, xacro)
@@ -25,5 +25,5 @@
     </joint>
   </xacro:macro>
-  <xacro:macro name="amazing_hand_command_joint" params="prefix name lower upper">
+  <xacro:macro name="amazing_hand_command_joint" params="prefix name lower upper initial:=0.0">
     <joint name="${prefix}${name}">
       <command_interface name="position">
@@ -31,5 +31,7 @@
         <param name="max">${upper}</param>
       </command_interface>
-      <state_interface name="position"/>
+      <state_interface name="position">
+        <param name="initial_value">${initial}</param>
+      </state_interface>
     </joint>
   </xacro:macro>

File: Open_arm_a1_ws/src/openarm_description/urdf/ee/amazing_hand/l_ahand.urdf (robot description, URDF)
Before this commit: robot left_hand, 123 links, 122 joints
Joints:
- joint cylindrical_1_1: mimic joint=j21 multiplier=-0.856286 offset=-0.038898 -> joint=j24 multiplier=-0.856286 offset=-0.038898
- joint cylindrical_1_3: mimic joint=j22 multiplier=-0.856286 offset=-0.038898 -> joint=j21 multiplier=-0.856286 offset=-0.038898
- joint cylindrical_1_7: mimic joint=j24 multiplier=-0.856286 offset=-0.038898 -> joint=j22 multiplier=-0.856286 offset=-0.038898
- joint revolute_1: mimic joint=j11 multiplier=1 offset=0 -> joint=j14 multiplier=1 offset=0
- joint revolute_1_1: mimic joint=j12 multiplier=1 offset=0 -> joint=j11 multiplier=1 offset=0
- joint revolute_1_4: mimic joint=j14 multiplier=1 offset=0 -> joint=j12 multiplier=1 offset=0
- joint revolute_2: mimic joint=j21 multiplier=-1.0 offset=0 -> joint=j24 multiplier=-1.0 offset=0
- joint revolute_2_1: mimic joint=j22 multiplier=-1.0 offset=0 -> joint=j21 multiplier=-1.0 offset=0
- joint revolute_2_3: mimic joint=j24 multiplier=-1.0 offset=0 -> joint=j22 multiplier=-1.0 offset=0
- joint revolute_3_1: mimic joint=j21 multiplier=1.062201 offset=-0.015673 -> joint=j24 multiplier=1.062201 offset=-0.015673; origin xyz=-0.0019 -7.63278e-17 -0.0095 rpy=-1.72061e-13 -1.80591e-16 1.19349e-15 -> xyz=-0.0019 0 -0.0095 rpy=0 0 0
- joint revolute_3_2: mimic joint=j22 multiplier=1.062201 offset=-0.015673 -> joint=j21 multiplier=1.062201 offset=-0.015673; origin xyz=-0.0019 0 -0.0095 rpy=-9.90587e-15 -6.09448e-17 3.97123e-16 -> xyz=-0.0019 0 -0.0095 rpy=0 0 0
- joint revolute_3_3: origin xyz=-0.0019 -5.55112e-17 -0.0095 rpy=-1.60716e-13 1.15478e-16 -3.33067e-16 -> xyz=-0.0019 0 -0.0095 rpy=0 0 0
- joint revolute_3_4: mimic joint=j24 multiplier=1.062201 offset=-0.015673 -> joint=j22 multiplier=1.062201 offset=-0.015673; origin xyz=-0.0019 -9.36751e-17 -0.0095 rpy=6.07431e-16 -9.9073e-16 2.56045e-15 -> xyz=-0.0019 0 -0.0095 rpy=0 0 0
- joint revolute_5: mimic joint=j21 multiplier=1.019021 offset=0.037525 -> joint=j24 multiplier=1.019021 offset=0.037525
- joint revolute_5_1: mimic joint=j22 multiplier=1.019021 offset=0.037525 -> joint=j21 multiplier=1.019021 offset=0.037525
- joint revolute_5_3: mimic joint=j24 multiplier=1.019021 offset=0.037525 -> joint=j22 multiplier=1.019021 offset=0.037525
- joint revolute_6: mimic joint=j21 multiplier=-1.019022 offset=-0.037525 -> joint=j24 multiplier=-1.019022 offset=-0.037525
- joint revolute_6_1: mimic joint=j22 multiplier=-1.019022 offset=-0.037525 -> joint=j21 multiplier=-1.019022 offset=-0.037525
- joint revolute_6_3: mimic joint=j24 multiplier=-1.019022 offset=-0.037525 -> joint=j22 multiplier=-1.019022 offset=-0.037525

File: Open_arm_a1_ws/src/openarm_description/urdf/ee/amazing_hand/l_ahand_macro.xacro (robot description, xacro)
@@ -1390,5 +1390,5 @@
         <parent link="${prefix}cylindrical_1" />
         <child link="${prefix}distal_2" />
-    <mimic joint="${prefix[:-6]}j21" multiplier="-0.856286" offset="-0.038898" /></joint>
+    <mimic joint="${prefix[:-6]}j24" multiplier="-0.856286" offset="-0.038898" /></joint>
     <joint name="${prefix}cylindrical_1_2" type="prismatic">
         <origin xyz="-0.00035 0.0496106 0.00943613" rpy="-0.0804909 5.31725e-17 -1.07388e-15" />
@@ -1403,5 +1403,5 @@
         <parent link="${prefix}cylindrical_1_1" />
         <child link="${prefix}distal_1" />
-    <mimic joint="${prefix[:-6]}j22" multiplier="-0.856286" offset="-0.038898" /></joint>
+    <mimic joint="${prefix[:-6]}j21" multiplier="-0.856286" offset="-0.038898" /></joint>
     <joint name="${prefix}cylindrical_1_4" type="prismatic">
         <origin xyz="-0.00035 0.0496106 0.00943613" rpy="-0.0804909 1.6886e-15 -1.81943e-15" />
@@ -1429,5 +1429,5 @@
         <parent link="${prefix}cylindrical_1_3" />
         <child link="${prefix}distal" />
-    <mimic joint="${prefix[:-6]}j24" multiplier="-0.856286" offset="-0.038898" /></joint>
+    <mimic joint="${prefix[:-6]}j22" multiplier="-0.856286" offset="-0.038898" /></joint>
     <joint name="${prefix}fastened_1" type="fixed">
         <origin xyz="0.00605 -0.01245 -0.008" rpy="1.5708 -1.12906e-14 3.14159" />
@@ -1664,5 +1664,5 @@
         <child link="${prefix}gimbal_2" />
         <limit effort="1" velocity="1" lower="-0.349066" upper="0.349066" />
-    <mimic joint="${prefix[:-6]}j11" multiplier="1" offset="0" /></joint>
+    <mimic joint="${prefix[:-6]}j14" multiplier="1" offset="0" /></joint>
     <joint name="${prefix}revolute_1_1" type="revolute">
         <origin xyz="-6.93889e-18 -6.93889e-18 0.001" rpy="-3.14159 2.05193e-27 4.1595e-14" />
@@ -1671,5 +1671,5 @@
         <child link="${prefix}gimbal_1" />
         <limit effort="1" velocity="1" lower="-0.349066" upper="0.349066" />
-    <mimic joint="${prefix[:-6]}j12" multiplier="1" offset="0" /></joint>
+    <mimic joint="${prefix[:-6]}j11" multiplier="1" offset="0" /></joint>
     <joint name="${prefix}revolute_1_2" type="revolute">
         <origin xyz="-9.02056e-17 -4.85723e-17 0.001" rpy="3.14159 -2.01489e-16 -6.93889e-16" />
@@ -1691,5 +1691,5 @@
         <child link="${prefix}gimbal" />
         <limit effort="1" velocity="1" lower="-0.349066" upper="0.349066" />
-    <mimic joint="${prefix[:-6]}j14" multiplier="1" offset="0" /></joint>
+    <mimic joint="${prefix[:-6]}j12" multiplier="1" offset="0" /></joint>
     <joint name="${prefix}revolute_2" type="revolute">
         <origin xyz="-0.00525 -1.73472e-17 -0.0035" rpy="-1.80303e-13 -9.84526e-17 1.69309e-15" />
@@ -1698,5 +1698,5 @@
         <child link="${prefix}proximal_2" />
         <limit effort="1" velocity="1" lower="-1.35615" upper="0.0924772" />
-    <mimic joint="${prefix[:-6]}j21" multiplier="-1.0" offset="0" /></joint>
+    <mimic joint="${prefix[:-6]}j24" multiplier="-1.0" offset="0" /></joint>
     <joint name="${prefix}revolute_2_1" type="revolute">
         <origin xyz="-0.00525 6.93889e-18 -0.0035" rpy="-1.60745e-14 -4.74371e-17 5.18347e-15" />
@@ -1705,5 +1705,5 @@
         <child link="${prefix}proximal_1" />
         <limit effort="1" velocity="1" lower="-1.35615" upper="0.0924772" />
-    <mimic joint="${prefix[:-6]}j22" multiplier="-1.0" offset="0" /></joint>
+    <mimic joint="${prefix[:-6]}j21" multiplier="-1.0" offset="0" /></joint>
     <joint name="${prefix}revolute_2_2" type="revolute">
         <origin xyz="-0.00525 -9.02056e-17 -0.0035" rpy="-1.69048e-13 2.00624e-17 3.60822e-16" />
@@ -1719,5 +1719,5 @@
         <child link="${prefix}proximal" />
         <limit effort="1" velocity="1" lower="-1.35615" upper="0.0924772" />
-    <mimic joint="${prefix[:-6]}j24" multiplier="-1.0" offset="0" /></joint>
+    <mimic joint="${prefix[:-6]}j22" multiplier="-1.0" offset="0" /></joint>
     <joint name="${prefix}revolute_2_4" type="continuous">
         <origin xyz="-0.00061573 -0.0150929 -0.003" rpy="-4.54497e-16 -6.24238e-16 1.5708" />
@@ -1733,17 +1733,17 @@
     </joint>
     <joint name="${prefix}revolute_3_1" type="continuous">
-        <origin xyz="-0.0019 -7.63278e-17 -0.0095" rpy="-1.72061e-13 -1.80591e-16 1.19349e-15" />
+        <origin xyz="-0.0019 0 -0.0095" rpy="0 0 0" />
         <axis xyz="-1 0 0" />
         <parent link="${prefix}gimbal_2" />
         <child link="${prefix}link_2" />
-    <mimic joint="${prefix[:-6]}j21" multiplier="1.062201" offset="-0.015673" /></joint>
+    <mimic joint="${prefix[:-6]}j24" multiplier="1.062201" offset="-0.015673" /></joint>
     <joint name="${prefix}revolute_3_2" type="continuous">
-        <origin xyz="-0.0019 0 -0.0095" rpy="-9.90587e-15 -6.09448e-17 3.97123e-16" />
+        <origin xyz="-0.0019 0 -0.0095" rpy="0 0 0" />
         <axis xyz="-1 0 0" />
         <parent link="${prefix}gimbal_1" />
         <child link="${prefix}link_1" />
-    <mimic joint="${prefix[:-6]}j22" multiplier="1.062201" offset="-0.015673" /></joint>
+    <mimic joint="${prefix[:-6]}j21" multiplier="1.062201" offset="-0.015673" /></joint>
     <joint name="${prefix}revolute_3_3" type="continuous">
-        <origin xyz="-0.0019 -5.55112e-17 -0.0095" rpy="-1.60716e-13 1.15478e-16 -3.33067e-16" />
+        <origin xyz="-0.0019 0 -0.0095" rpy="0 0 0" />
         <axis xyz="-1 0 0" />
         <parent link="${prefix}gimbal_3" />
@@ -1751,9 +1751,9 @@
     <mimic joint="${prefix[:-6]}j23" multiplier="1.062201" offset="-0.015673" /></joint>
     <joint name="${prefix}revolute_3_4" type="continuous">
-        <origin xyz="-0.0019 -9.36751e-17 -0.0095" rpy="6.07431e-16 -9.9073e-16 2.56045e-15" />
+        <origin xyz="-0.0019 0 -0.0095" rpy="0 0 0" />
         <axis xyz="-1 0 0" />
         <parent link="${prefix}gimbal" />
         <child link="${prefix}link" />
-    <mimic joint="${prefix[:-6]}j24" multiplier="1.062201" offset="-0.015673" /></joint>
+    <mimic joint="${prefix[:-6]}j22" multiplier="1.062201" offset="-0.015673" /></joint>
     <joint name="${prefix}revolute_4" type="continuous">
         <origin xyz="-0.0270789 -0.0251197 -0.003" rpy="1.44071e-15 1.72452e-16 -3.3285e-16" />
@@ -1792,5 +1792,5 @@
         <child link="${prefix}custom_servo_horn_5" />
         <limit effort="1" velocity="1" lower="-2.18166" upper="0.959931" />
-    <mimic joint="${prefix[:-6]}j21" multiplier="1.019021" offset="0.037525" /></joint>
+    <mimic joint="${prefix[:-6]}j24" multiplier="1.019021" offset="0.037525" /></joint>
     <joint name="${prefix}revolute_5_1" type="revolute">
         <origin xyz="-6.93889e-18 -0.0087 -0.01995" rpy="1.5708 -1.55931e-13 -2.47818e-16" />
@@ -1799,5 +1799,5 @@
         <child link="${prefix}custom_servo_horn_2" />
         <limit effort="1" velocity="1" lower="-2.18166" upper="0.959931" />
-    <mimic joint="${prefix[:-6]}j22" multiplier="1.019021" offset="0.037525" /></joint>
+    <mimic joint="${prefix[:-6]}j21" multiplier="1.019021" offset="0.037525" /></joint>
     <joint name="${prefix}revolute_5_2" type="revolute">
         <origin xyz="-8.67362e-18 -0.0087 -0.01995" rpy="1.5708 8.76862e-15 -1.40489e-14" />
@@ -1813,5 +1813,5 @@
         <child link="${prefix}custom_servo_horn" />
         <limit effort="1" velocity="1" lower="-2.18166" upper="0.959931" />
-    <mimic joint="${prefix[:-6]}j24" multiplier="1.019021" offset="0.037525" /></joint>
+    <mimic joint="${prefix[:-6]}j22" multiplier="1.019021" offset="0.037525" /></joint>
     <joint name="${prefix}revolute_6" type="revolute">
         <origin xyz="-2.08167e-17 -0.0087 -0.01995" rpy="-1.5708 1.54195e-15 3.14159" />
@@ -1820,5 +1820,5 @@
         <child link="${prefix}custom_servo_horn_4" />
         <limit effort="1" velocity="1" lower="-0.959931" upper="2.18166" />
-    <mimic joint="${prefix[:-6]}j21" multiplier="-1.019022" offset="-0.037525" /></joint>
+    <mimic joint="${prefix[:-6]}j24" multiplier="-1.019022" offset="-0.037525" /></joint>
     <joint name="${prefix}revolute_6_1" type="revolute">
         <origin xyz="-2.77556e-17 -0.0087 -0.01995" rpy="-1.5708 2.88658e-15 3.14159" />
@@ -1827,5 +1827,5 @@
         <child link="${prefix}custom_servo_horn_3" />
         <limit effort="1" velocity="1" lower="-0.959931" upper="2.18166" />
-    <mimic joint="${prefix[:-6]}j22" multiplier="-1.019022" offset="-0.037525" /></joint>
+    <mimic joint="${prefix[:-6]}j21" multiplier="-1.019022" offset="-0.037525" /></joint>
     <joint name="${prefix}revolute_6_2" type="revolute">
         <origin xyz="-1.34441e-17 -0.0087 -0.01995" rpy="-1.5708 -2.06903e-17 3.14159" />
@@ -1841,5 +1841,5 @@
         <child link="${prefix}custom_servo_horn_1" />
         <limit effort="1" velocity="1" lower="-0.959931" upper="2.18166" />
-    <mimic joint="${prefix[:-6]}j24" multiplier="-1.019022" offset="-0.037525" /></joint>
+    <mimic joint="${prefix[:-6]}j22" multiplier="-1.019022" offset="-0.037525" /></joint>
   </xacro:macro>
 </robot>

File: Open_arm_a1_ws/src/openarm_description/urdf/ee/amazing_hand/r_ahand.urdf (robot description, URDF)
Before this commit: robot right_hand, 123 links, 122 joints
Joints:
- joint cylindrical_1_1: mimic joint=j21 multiplier=0.893781 offset=0.027842 -> joint=j24 multiplier=0.893781 offset=0.027842
- joint cylindrical_1_3: mimic joint=j22 multiplier=0.893781 offset=0.027842 -> joint=j21 multiplier=0.893781 offset=0.027842
- joint cylindrical_1_7: mimic joint=j24 multiplier=0.893781 offset=0.027842 -> joint=j22 multiplier=0.893781 offset=0.027842
- joint revolute_1: mimic joint=j11 multiplier=1 offset=0 -> joint=j14 multiplier=1 offset=0
- joint revolute_1_1: mimic joint=j12 multiplier=1 offset=0 -> joint=j11 multiplier=1 offset=0
- joint revolute_1_4: mimic joint=j14 multiplier=1 offset=0 -> joint=j12 multiplier=1 offset=0
- joint revolute_2: mimic joint=j21 multiplier=1.0 offset=0 -> joint=j24 multiplier=1.0 offset=0
- joint revolute_2_1: mimic joint=j22 multiplier=1.0 offset=0 -> joint=j21 multiplier=1.0 offset=0
- joint revolute_2_3: mimic joint=j24 multiplier=1.0 offset=0 -> joint=j22 multiplier=1.0 offset=0
- joint revolute_3_1: mimic joint=j21 multiplier=-1.071506 offset=0.018398 -> joint=j24 multiplier=-1.071506 offset=0.018398; origin xyz=0.0019 -7.63278e-17 -0.0095 rpy=-1.72061e-13 1.80591e-16 -1.19349e-15 -> xyz=0.0019 0 -0.0095 rpy=0 0 0
- joint revolute_3_2: mimic joint=j22 multiplier=-1.071506 offset=0.018398 -> joint=j21 multiplier=-1.071506 offset=0.018398; origin xyz=0.0019 0 -0.0095 rpy=-9.90587e-15 6.09448e-17 -3.97123e-16 -> xyz=0.0019 0 -0.0095 rpy=0 0 0
- joint revolute_3_3: origin xyz=0.0019 -5.55112e-17 -0.0095 rpy=-1.60716e-13 -1.15478e-16 3.33067e-16 -> xyz=0.0019 0 -0.0095 rpy=0 0 0
- joint revolute_3_4: mimic joint=j24 multiplier=-1.071506 offset=0.018398 -> joint=j22 multiplier=-1.071506 offset=0.018398; origin xyz=0.0019 -9.36751e-17 -0.0095 rpy=6.07431e-16 9.9073e-16 -2.56045e-15 -> xyz=0.0019 0 -0.0095 rpy=0 0 0
- joint revolute_5: mimic joint=j21 multiplier=-1.390791 offset=0.071818 -> joint=j24 multiplier=-1.390791 offset=0.071818
- joint revolute_5_1: mimic joint=j22 multiplier=-1.390791 offset=0.071818 -> joint=j21 multiplier=-1.390791 offset=0.071818
- joint revolute_5_3: mimic joint=j24 multiplier=-1.390791 offset=0.071818 -> joint=j22 multiplier=-1.390791 offset=0.071818
- joint revolute_6: mimic joint=j21 multiplier=1.390793 offset=-0.071819 -> joint=j24 multiplier=1.390793 offset=-0.071819
- joint revolute_6_1: mimic joint=j22 multiplier=1.390793 offset=-0.071819 -> joint=j21 multiplier=1.390793 offset=-0.071819
- joint revolute_6_3: mimic joint=j24 multiplier=1.390793 offset=-0.071819 -> joint=j22 multiplier=1.390793 offset=-0.071819
