Commit message: Fix joint references and update arm base positions in URDF files
- Updated mimic joint references in left and right hand URDF and XACRO files to correct joint mappings.
- Adjusted the base position and orientation parameters for the right and left arms in the robot's main XACRO file to ensure proper alignment.

File: Open_arm_a1_ws/src/openarm_description/urdf/ee/amazing_hand/r_ahand_macro.xacro (robot description, xacro)
@@ -1390,5 +1390,5 @@
         <parent link="${prefix}cylindrical_1" />
         <child link="${prefix}distal_2" />
-    <mimic joint="${prefix[:-6]}j21" multiplier="0.893781" offset="0.027842" /></joint>
+    <mimic joint="${prefix[:-6]}j24" multiplier="0.893781" offset="0.027842" /></joint>
     <joint name="${prefix}cylindrical_1_2" type="prismatic">
         <origin xyz="0.00035 0.0496106 0.00943613" rpy="-0.0804909 -5.31725e-17 1.07388e-15" />
@@ -1403,5 +1403,5 @@
         <parent link="${prefix}cylindrical_1_1" />
         <child link="${prefix}distal_1" />
-    <mimic joint="${prefix[:-6]}j22" multiplier="0.893781" offset="0.027842" /></joint>
+    <mimic joint="${prefix[:-6]}j21" multiplier="0.893781" offset="0.027842" /></joint>
     <joint name="${prefix}cylindrical_1_4" type="prismatic">
         <origin xyz="0.00035 0.0496106 0.00943613" rpy="-0.0804909 -1.6886e-15 1.81943e-15" />
@@ -1429,5 +1429,5 @@
         <parent link="${prefix}cylindrical_1_3" />
         <child link="${prefix}distal" />
-    <mimic joint="${prefix[:-6]}j24" multiplier="0.893781" offset="0.027842" /></joint>
+    <mimic joint="${prefix[:-6]}j22" multiplier="0.893781" offset="0.027842" /></joint>
     <joint name="${prefix}fastened_1" type="fixed">
         <origin xyz="-0.00605 -0.01245 -0.008" rpy="1.5708 1.12906e-14 -3.14159" />
@@ -1664,5 +1664,5 @@
         <child link="${prefix}gimbal_2" />
         <limit effort="1" velocity="1" lower="-0.349066" upper="0.349066" />
-    <mimic joint="${prefix[:-6]}j11" multiplier="1" offset="0" /></joint>
+    <mimic joint="${prefix[:-6]}j14" multiplier="1" offset="0" /></joint>
     <joint name="${prefix}revolute_1_1" type="revolute">
         <origin xyz="6.93889e-18 -6.93889e-18 0.001" rpy="-3.14159 -2.05193e-27 -4.1595e-14" />
@@ -1671,5 +1671,5 @@
         <child link="${prefix}gimbal_1" />
         <limit effort="1" velocity="1" lower="-0.349066" upper="0.349066" />
-    <mimic joint="${prefix[:-6]}j12" multiplier="1" offset="0" /></joint>
+    <mimic joint="${prefix[:-6]}j11" multiplier="1" offset="0" /></joint>
     <joint name="${prefix}revolute_1_2" type="revolute">
         <origin xyz="9.02056e-17 -4.85723e-17 0.001" rpy="3.14159 2.01489e-16 6.93889e-16" />
@@ -1691,5 +1691,5 @@
         <child link="${prefix}gimbal" />
         <limit effort="1" velocity="1" lower="-0.349066" upper="0.349066" />
-    <mimic joint="${prefix[:-6]}j14" multiplier="1" offset="0" /></joint>
+    <mimic joint="${prefix[:-6]}j12" multiplier="1" offset="0" /></joint>
     <joint name="${prefix}revolute_2" type="revolute">
         <origin xyz="0.00525 -1.73472e-17 -0.0035" rpy="-1.80303e-13 9.84526e-17 -1.69309e-15" />
@@ -1698,5 +1698,5 @@
         <child link="${prefix}proximal_2" />
         <limit effort="1" velocity="1" lower="-0.0924772" upper="1.35615" />
-    <mimic joint="${prefix[:-6]}j21" multiplier="1.0" offset="0" /></joint>
+    <mimic joint="${prefix[:-6]}j24" multiplier="1.0" offset="0" /></joint>
     <joint name="${prefix}revolute_2_1" type="revolute">
         <origin xyz="0.00525 6.93889e-18 -0.0035" rpy="-1.60745e-14 4.74371e-17 -5.18347e-15" />
@@ -1705,5 +1705,5 @@
         <child link="${prefix}proximal_1" />
         <limit effort="1" velocity="1" lower="-0.0924772" upper="1.35615" />
-    <mimic joint="${prefix[:-6]}j22" multiplier="1.0" offset="0" /></joint>
+    <mimic joint="${prefix[:-6]}j21" multiplier="1.0" offset="0" /></joint>
     <joint name="${prefix}revolute_2_2" type="revolute">
         <origin xyz="0.00525 -9.02056e-17 -0.0035" rpy="-1.69048e-13 -2.00624e-17 -3.60822e-16" />
@@ -1719,5 +1719,5 @@
         <child link="${prefix}proximal" />
         <limit effort="1" velocity="1" lower="-0.0924772" upper="1.35615" />
-    <mimic joint="${prefix[:-6]}j24" multiplier="1.0" offset="0" /></joint>
+    <mimic joint="${prefix[:-6]}j22" multiplier="1.0" offset="0" /></joint>
     <joint name="${prefix}revolute_2_4" type="continuous">
         <origin xyz="0.00061573 -0.0150929 -0.003" rpy="-4.54497e-16 6.24238e-16 -1.5708" />
@@ -1733,17 +1733,17 @@
     </joint>
     <joint name="${prefix}revolute_3_1" type="continuous">
-        <origin xyz="0.0019 -7.63278e-17 -0.0095" rpy="-1.72061e-13 1.80591e-16 -1.19349e-15" />
+        <origin xyz="0.0019 0 -0.0095" rpy="0 0 0" />
         <axis xyz="1 0 0" />
         <parent link="${prefix}gimbal_2" />
         <child link="${prefix}link_2" />
-    <mimic joint="${prefix[:-6]}j21" multiplier="-1.071506" offset="0.018398" /></joint>
+    <mimic joint="${prefix[:-6]}j24" multiplier="-1.071506" offset="0.018398" /></joint>
     <joint name="${prefix}revolute_3_2" type="continuous">
-        <origin xyz="0.0019 0 -0.0095" rpy="-9.90587e-15 6.09448e-17 -3.97123e-16" />
+        <origin xyz="0.0019 0 -0.0095" rpy="0 0 0" />
         <axis xyz="1 0 0" />
         <parent link="${prefix}gimbal_1" />
         <child link="${prefix}link_1" />
-    <mimic joint="${prefix[:-6]}j22" multiplier="-1.071506" offset="0.018398" /></joint>
+    <mimic joint="${prefix[:-6]}j21" multiplier="-1.071506" offset="0.018398" /></joint>
     <joint name="${prefix}revolute_3_3" type="continuous">
-        <origin xyz="0.0019 -5.55112e-17 -0.0095" rpy="-1.60716e-13 -1.15478e-16 3.33067e-16" />
+        <origin xyz="0.0019 0 -0.0095" rpy="0 0 0" />
         <axis xyz="1 0 0" />
         <parent link="${prefix}gimbal_3" />
@@ -1751,9 +1751,9 @@
     <mimic joint="${prefix[:-6]}j23" multiplier="-1.071506" offset="0.018398" /></joint>
     <joint name="${prefix}revolute_3_4" type="continuous">
-        <origin xyz="0.0019 -9.36751e-17 -0.0095" rpy="6.07431e-16 9.9073e-16 -2.56045e-15" />
+        <origin xyz="0.0019 0 -0.0095" rpy="0 0 0" />
         <axis xyz="1 0 0" />
         <parent link="${prefix}gimbal" />
         <child link="${prefix}link" />
-    <mimic joint="${prefix[:-6]}j24" multiplier="-1.071506" offset="0.018398" /></joint>
+    <mimic joint="${prefix[:-6]}j22" multiplier="-1.071506" offset="0.018398" /></joint>
     <joint name="${prefix}revolute_4" type="continuous">
         <origin xyz="0.0270789 -0.0251197 -0.003" rpy="1.44071e-15 -1.72452e-16 3.3285e-16" />
@@ -1792,5 +1792,5 @@
         <child link="${prefix}custom_servo_horn_5" />
         <limit effort="1" velocity="1" lower="-2.18166" upper="0.959931" />
-    <mimic joint="${prefix[:-6]}j21" multiplier="-1.390791" offset="0.071818" /></joint>
+    <mimic joint="${prefix[:-6]}j24" multiplier="-1.390791" offset="0.071818" /></joint>
     <joint name="${prefix}revolute_5_1" type="revolute">
         <origin xyz="6.93889e-18 -0.0087 -0.01995" rpy="1.5708 1.55931e-13 2.47818e-16" />
@@ -1799,5 +1799,5 @@
         <child link="${prefix}custom_servo_horn_2" />
         <limit effort="1" velocity="1" lower="-2.18166" upper="0.959931" />
-    <mimic joint="${prefix[:-6]}j22" multiplier="-1.390791" offset="0.071818" /></joint>
+    <mimic joint="${prefix[:-6]}j21" multiplier="-1.390791" offset="0.071818" /></joint>
     <joint name="${prefix}revolute_5_2" type="revolute">
         <origin xyz="8.67362e-18 -0.0087 -0.01995" rpy="1.5708 -8.76862e-15 1.40489e-14" />
@@ -1813,5 +1813,5 @@
         <child link="${prefix}custom_servo_horn" />
         <limit effort="1" velocity="1" lower="-2.18166" upper="0.959931" />
-    <mimic joint="${prefix[:-6]}j24" multiplier="-1.390791" offset="0.071818" /></joint>
+    <mimic joint="${prefix[:-6]}j22" multiplier="-1.390791" offset="0.071818" /></joint>
     <joint name="${prefix}revolute_6" type="revolute">
         <origin xyz="2.08167e-17 -0.0087 -0.01995" rpy="-1.5708 -1.54195e-15 -3.14159" />
@@ -1820,5 +1820,5 @@
         <child link="${prefix}custom_servo_horn_4" />
         <limit effort="1" velocity="1" lower="-0.959931" upper="2.18166" />
-    <mimic joint="${prefix[:-6]}j21" multiplier="1.390793" offset="-0.071819" /></joint>
+    <mimic joint="${prefix[:-6]}j24" multiplier="1.390793" offset="-0.071819" /></joint>
     <joint name="${prefix}revolute_6_1" type="revolute">
         <origin xyz="2.77556e-17 -0.0087 -0.01995" rpy="-1.5708 -2.88658e-15 -3.14159" />
@@ -1827,5 +1827,5 @@
         <child link="${prefix}custom_servo_horn_3" />
         <limit effort="1" velocity="1" lower="-0.959931" upper="2.18166" />
-    <mimic joint="${prefix[:-6]}j22" multiplier="1.390793" offset="-0.071819" /></joint>
+    <mimic joint="${prefix[:-6]}j21" multiplier="1.390793" offset="-0.071819" /></joint>
     <joint name="${prefix}revolute_6_2" type="revolute">
         <origin xyz="1.34441e-17 -0.0087 -0.01995" rpy="-1.5708 2.06903e-17 -3.14159" />
@@ -1841,5 +1841,5 @@
         <child link="${prefix}custom_servo_horn_1" />
         <limit effort="1" velocity="1" lower="-0.959931" upper="2.18166" />
-    <mimic joint="${prefix[:-6]}j24" multiplier="1.390793" offset="-0.071819" /></joint>
+    <mimic joint="${prefix[:-6]}j22" multiplier="1.390793" offset="-0.071819" /></joint>
   </xacro:macro>
 </robot>

File: Open_arm_a1_ws/src/openarm_description/urdf/robot/v10.urdf.xacro (robot description, xacro)
@@ -23,8 +23,8 @@
   <xacro:arg name="fake_sensor_commands" default="false" />
   <xacro:arg name="bimanual" default="false" />
-  <xacro:arg name="right_arm_base_xyz" default="-0.03 0.118 0.21" />
-  <xacro:arg name="right_arm_base_rpy" default="1.5708 0 3.14159" />
-  <xacro:arg name="left_arm_base_xyz" default="-0.03 -0.112 0.21" />
-  <xacro:arg name="left_arm_base_rpy" default="-1.5708 0 3.14159" />
+  <xacro:arg name="right_arm_base_xyz" default="-0.03 -0.118 0.21" />
+  <xacro:arg name="right_arm_base_rpy" default="-1.5708 3.14159 3.14159" />
+  <xacro:arg name="left_arm_base_xyz" default="-0.03 0.112 0.21" />
+  <xacro:arg name="left_arm_base_rpy" default="1.5708 3.14159 3.14159" />
   <xacro:arg name="can_fd" default="true" />
   <xacro:arg name="gazebo" default="false" />

Commit message: add head sequence

File: Open_arm_a1_ws/src/openarm_description/urdf/body/openarm_body.xacro (robot description, xacro)
@@ -109,5 +109,5 @@
         <child link="${prefix}neck_link" />
         <axis xyz="0 0 -1" />
-        <limit lower="-1.57" upper="1.57" effort="10" velocity="3" />
+        <limit lower="-1.0472" upper="1.0472" effort="10" velocity="3" />
       </joint>
       <link name="${prefix}head_link">
@@ -138,5 +138,5 @@
         <child link="${prefix}head_link" />
         <axis xyz="0.034355 -0.034358 0.99882" />
-        <limit lower="-1.57" upper="1.57" effort="10" velocity="3" />
+        <limit lower="-1.0472" upper="1.0472" effort="10" velocity="3" />
       </joint>
       <!-- Cosmetic outer shell, visual-only (no collision geometry, doesn't
