Commit message: feat: update BehaviorTree.ROS2 implementation and refine topic-based control and MoveIt configuration.

File: Open_arm_a1_ws/src/openarm_description/urdf/robot/openarm_robot.xacro (robot description, xacro)
@@ -22,4 +22,5 @@
             can_interface:=''
             use_fake_hardware:=false
+            use_isaac_sim:=false
             fake_sensor_commands:=false
             no_prefix:='false'
@@ -118,4 +119,5 @@
             right_can_interface="${right_can_interface}"
             use_fake_hardware="${use_fake_hardware}"
+            use_isaac_sim="${use_isaac_sim}"
             fake_sensor_commands="${fake_sensor_commands}"
             left_arm_prefix="${left_arm_prefix}"

File: Open_arm_a1_ws/src/openarm_description/urdf/robot/v10.urdf.xacro (robot description, xacro)
@@ -20,4 +20,5 @@
   <xacro:arg name="right_arm_prefix" default="right_" />
   <xacro:arg name="use_fake_hardware" default="false" />
+  <xacro:arg name="use_isaac_sim" default="false" />
   <xacro:arg name="fake_sensor_commands" default="false" />
   <xacro:arg name="bimanual" default="false" />
@@ -56,4 +57,5 @@
   right_arm_prefix="$(arg right_arm_prefix)"
   use_fake_hardware="$(arg use_fake_hardware)"
+  use_isaac_sim="$(arg use_isaac_sim)"
   fake_sensor_commands="$(arg fake_sensor_commands)"
   no_prefix="$(arg no_prefix)"

File: Open_arm_a1_ws/src/openarm_description/urdf/ros2_control/openarm.bimanual.ros2_control.xacro (robot description, xacro)
@@ -7,4 +7,5 @@
              right_can_interface:=^|can0
              use_fake_hardware:=^|false
+             use_isaac_sim:=^|false
              fake_sensor_commands:=^|false
              hand:=^|false
@@ -16,29 +17,36 @@
         <hardware>
           <param name="arm_type">${arm_type}</param>
-          <xacro:if value="${use_fake_hardware}">
-            <plugin>mock_components/GenericSystem</plugin>
-            <param name="fake_sensor_commands">${fake_sensor_commands}</param>
-            <param name="state_following_offset">0.0</param>
+          <xacro:if value="${use_isaac_sim}">
+            <plugin>topic_based_ros2_control/TopicBasedSystem</plugin>
+            <param name="joint_commands_topic">/isaac_left_arm/joint_commands</param>
+            <param name="joint_states_topic">/isaac_left_arm/joint_states</param>
           </xacro:if>
-          <xacro:unless value="${use_fake_hardware}">
-            <plugin>openarm_hardware/OpenArm_v10HW</plugin>
-            <param name="can_interface">${left_can_interface}</param>
-            <param name="arm_prefix">${left_arm_prefix}</param>
-            <param name="hand">${hand}</param>
-            <param name="can_fd">${can_fd}</param>
-            <param name="kp1">${control_gains['joint1']['kp']}</param>
-            <param name="kp2">${control_gains['joint2']['kp']}</param>
-            <param name="kp3">${control_gains['joint3']['kp']}</param>
-            <param name="kp4">${control_gains['joint4']['kp']}</param>
-            <param name="kp5">${control_gains['joint5']['kp']}</param>
-            <param name="kp6">${control_gains['joint6']['kp']}</param>
-            <param name="kp7">${control_gains['joint7']['kp']}</param>
-            <param name="kd1">${control_gains['joint1']['kd']}</param>
-            <param name="kd2">${control_gains['joint2']['kd']}</param>
-            <param name="kd3">${control_gains['joint3']['kd']}</param>
-            <param name="kd4">${control_gains['joint4']['kd']}</param>
-            <param name="kd5">${control_gains['joint5']['kd']}</param>
-            <param name="kd6">${control_gains['joint6']['kd']}</param>
-            <param name="kd7">${control_gains['joint7']['kd']}</param>
+          <xacro:unless value="${use_isaac_sim}">
+            <xacro:if value="${use_fake_hardware}">
+              <plugin>mock_components/GenericSystem</plugin>
+              <param name="fake_sensor_commands">${fake_sensor_commands}</param>
+              <param name="state_following_offset">0.0</param>
+            </xacro:if>
+            <xacro:unless value="${use_fake_hardware}">
+              <plugin>openarm_hardware/OpenArm_v10HW</plugin>
+              <param name="can_interface">${left_can_interface}</param>
+              <param name="arm_prefix">${left_arm_prefix}</param>
+              <param name="hand">${hand}</param>
+              <param name="can_fd">${can_fd}</param>
+              <param name="kp1">${control_gains['joint1']['kp']}</param>
+              <param name="kp2">${control_gains['joint2']['kp']}</param>
+              <param name="kp3">${control_gains['joint3']['kp']}</param>
+              <param name="kp4">${control_gains['joint4']['kp']}</param>
+              <param name="kp5">${control_gains['joint5']['kp']}</param>
+              <param name="kp6">${control_gains['joint6']['kp']}</param>
+              <param name="kp7">${control_gains['joint7']['kp']}</param>
+              <param name="kd1">${control_gains['joint1']['kd']}</param>
+              <param name="kd2">${control_gains['joint2']['kd']}</param>
+              <param name="kd3">${control_gains['joint3']['kd']}</param>
+              <param name="kd4">${control_gains['joint4']['kd']}</param>
+              <param name="kd5">${control_gains['joint5']['kd']}</param>
+              <param name="kd6">${control_gains['joint6']['kd']}</param>
+              <param name="kd7">${control_gains['joint7']['kd']}</param>
+            </xacro:unless>
           </xacro:unless>
         </hardware>
@@ -68,4 +76,19 @@
       <xacro:if value="${hand}">
         <xacro:configure_joint joint_name="openarm_${left_arm_prefix}finger_joint1" initial_position="0.0" />
+        <xacro:if value="${use_isaac_sim}">
+          <joint name="openarm_${left_arm_prefix}finger_joint2">
+            <param name="mimic">openarm_${left_arm_prefix}finger_joint1</param>
+            <param name="multiplier">1.0</param>
+            <state_interface name="position">
+              <param name="initial_value">0.0</param>
+            </state_interface>
+            <state_interface name="velocity">
+              <param name="initial_value">0.0</param>
+            </state_interface>
+            <state_interface name="effort">
+              <param name="initial_value">0.0</param>
+            </state_interface>
+          </joint>
+        </xacro:if>
       </xacro:if>
     </ros2_control>
@@ -74,29 +97,36 @@
         <hardware>
           <param name="arm_type">${arm_type}</param>
-          <xacro:if value="${use_fake_hardware}">
-            <plugin>mock_components/GenericSystem</plugin>
-            <param name="fake_sensor_commands">${fake_sensor_commands}</param>
-            <param name="state_following_offset">0.0</param>
+          <xacro:if value="${use_isaac_sim}">
+            <plugin>topic_based_ros2_control/TopicBasedSystem</plugin>
+            <param name="joint_commands_topic">/isaac_right_arm/joint_commands</param>
+            <param name="joint_states_topic">/isaac_right_arm/joint_states</param>
           </xacro:if>
-          <xacro:unless value="${use_fake_hardware}">
-            <plugin>openarm_hardware/OpenArm_v10HW</plugin>
-            <param name="can_interface">${right_can_interface}</param>
-            <param name="arm_prefix">${right_arm_prefix}</param>
-            <param name="hand">${hand}</param>
-            <param name="can_fd">${can_fd}</param>
-            <param name="kp1">${control_gains['joint1']['kp']}</param>
-            <param name="kp2">${control_gains['joint2']['kp']}</param>
-            <param name="kp3">${control_gains['joint3']['kp']}</param>
-            <param name="kp4">${control_gains['joint4']['kp']}</param>
-            <param name="kp5">${control_gains['joint5']['kp']}</param>
-            <param name="kp6">${control_gains['joint6']['kp']}</param>
-            <param name="kp7">${control_gains['joint7']['kp']}</param>
-            <param name="kd1">${control_gains['joint1']['kd']}</param>
-            <param name="kd2">${control_gains['joint2']['kd']}</param>
-            <param name="kd3">${control_gains['joint3']['kd']}</param>
-            <param name="kd4">${control_gains['joint4']['kd']}</param>
-            <param name="kd5">${control_gains['joint5']['kd']}</param>
-            <param name="kd6">${control_gains['joint6']['kd']}</param>
-            <param name="kd7">${control_gains['joint7']['kd']}</param>
+          <xacro:unless value="${use_isaac_sim}">
+            <xacro:if value="${use_fake_hardware}">
+              <plugin>mock_components/GenericSystem</plugin>
+              <param name="fake_sensor_commands">${fake_sensor_commands}</param>
+              <param name="state_following_offset">0.0</param>
+            </xacro:if>
+            <xacro:unless value="${use_fake_hardware}">
+              <plugin>openarm_hardware/OpenArm_v10HW</plugin>
+              <param name="can_interface">${right_can_interface}</param>
+              <param name="arm_prefix">${right_arm_prefix}</param>
+              <param name="hand">${hand}</param>
+              <param name="can_fd">${can_fd}</param>
+              <param name="kp1">${control_gains['joint1']['kp']}</param>
+              <param name="kp2">${control_gains['joint2']['kp']}</param>
+              <param name="kp3">${control_gains['joint3']['kp']}</param>
+              <param name="kp4">${control_gains['joint4']['kp']}</param>
+              <param name="kp5">${control_gains['joint5']['kp']}</param>
+              <param name="kp6">${control_gains['joint6']['kp']}</param>
+              <param name="kp7">${control_gains['joint7']['kp']}</param>
+              <param name="kd1">${control_gains['joint1']['kd']}</param>
+              <param name="kd2">${control_gains['joint2']['kd']}</param>
+              <param name="kd3">${control_gains['joint3']['kd']}</param>
+              <param name="kd4">${control_gains['joint4']['kd']}</param>
+              <param name="kd5">${control_gains['joint5']['kd']}</param>
+              <param name="kd6">${control_gains['joint6']['kd']}</param>
+              <param name="kd7">${control_gains['joint7']['kd']}</param>
+            </xacro:unless>
           </xacro:unless>
         </hardware>
@@ -110,4 +140,19 @@
       <xacro:if value="${hand}">
         <xacro:configure_joint joint_name="openarm_${right_arm_prefix}finger_joint1" initial_position="0.0" />
+        <xacro:if value="${use_isaac_sim}">
+          <joint name="openarm_${right_arm_prefix}finger_joint2">
+            <param name="mimic">openarm_${right_arm_prefix}finger_joint1</param>
+            <param name="multiplier">1.0</param>
+            <state_interface name="position">
+              <param name="initial_value">0.0</param>
+            </state_interface>
+            <state_interface name="velocity">
+              <param name="initial_value">0.0</param>
+            </state_interface>
+            <state_interface name="effort">
+              <param name="initial_value">0.0</param>
+            </state_interface>
+          </joint>
+        </xacro:if>
       </xacro:if>
     </ros2_control>
