Commit message: Add amazing hand support to openarm robot description
- Introduced new Xacro file for amazing hand arguments to define connection and offset parameters.
- Updated openarm_robot.xacro to include amazing hand macros for both left and right hands.
- Enhanced ROS2 control configurations to accommodate amazing hand integration, including joint commands and states.
- Modified bimanual and single arm control files to conditionally include amazing hand logic based on the specified end-effector type.

File: Open_arm_a1_ws/src/openarm_description/urdf/robot/openarm_robot.xacro (robot description, xacro)
@@ -56,4 +56,6 @@
     <xacro:include filename="$(find openarm_description)/urdf/ee/openarm_hand.xacro" />
     <xacro:include filename="$(find openarm_description)/urdf/ee/openarm_hand_macro.xacro" />
+    <xacro:include filename="$(find openarm_description)/urdf/ee/amazing_hand/r_ahand_macro.xacro" />
+    <xacro:include filename="$(find openarm_description)/urdf/ee/amazing_hand/l_ahand_macro.xacro" />
     <xacro:include filename="$(find openarm_description)/urdf/ros2_control/openarm.ros2_control.xacro" />
     <xacro:include filename="$(find openarm_description)/urdf/ros2_control/openarm.bimanual.ros2_control.xacro" />
@@ -125,5 +127,6 @@
             right_arm_prefix="${right_arm_prefix}"
             gazebo="${gazebo}"
-            hand="${hand}"/>
+            hand="${hand}"
+            ee_type="${ee_type}"/>
         </xacro:if>
         <xacro:if value="$(eval hand and ee_type == 'openarm_hand')">
@@ -155,4 +158,51 @@
             />
           </xacro:if>
+        <xacro:if value="$(eval hand and ee_type == 'amazing_hand')">
+            <xacro:amazing_hand_left
+                connected_to="openarm_left_link7"
+                prefix="openarm_left_ahand_"
+                xyz="$(arg xyz_ee)"
+                rpy="$(arg rpy_ee)"
+            />
+            <xacro:amazing_hand_right
+                connected_to="openarm_right_link7"
+                prefix="openarm_right_ahand_"
+                xyz="$(arg xyz_ee)"
+                rpy="$(arg rpy_ee)"
+            />
+            <!-- left_arm/right_arm MoveIt groups (defined once, shared across
+                 ee_type values) chain to openarm_<side>_hand_tcp regardless of
+                 which hand is attached; openarm_hand's own macro creates that
+                 link itself, so amazing_hand must too. Placed at the hand's
+                 mount point (same placeholder-calibration caveat as xyz_ee/
+                 rpy_ee above, not the true fingertip/grasp frame). -->
+            <link name="openarm_left_hand_tcp" />
+            <joint name="openarm_left_ahand_tcp_joint" type="fixed">
+                <origin xyz="0 0 0" rpy="0 0 0" />
+                <parent link="openarm_left_ahand_root" />
+                <child link="openarm_left_hand_tcp" />
+            </joint>
+            <link name="openarm_right_hand_tcp" />
+            <joint name="openarm_right_ahand_tcp_joint" type="fixed">
+                <origin xyz="0 0 0" rpy="0 0 0" />
+                <parent link="openarm_right_ahand_root" />
+                <child link="openarm_right_hand_tcp" />
+            </joint>
+            <xacro:if value="${ros2_control}">
+                <xacro:include filename="$(find openarm_description)/urdf/ee/amazing_hand/ahand.ros2_control.xacro" />
+                <xacro:amazing_hand_ros2_control
+                    prefix="openarm_left_"
+                    link_prefix="openarm_left_ahand_"
+                    joint_commands_topic="/left_ahand/joint_commands"
+                    joint_states_topic="/left_ahand/joint_states"
+                />
+                <xacro:amazing_hand_ros2_control
+                    prefix="openarm_right_"
+                    link_prefix="openarm_right_ahand_"
+                    joint_commands_topic="/right_ahand/joint_commands"
+                    joint_states_topic="/right_ahand/joint_states"
+                />
+            </xacro:if>
+        </xacro:if>
     </xacro:if>
     <xacro:if value="${not bimanual}">
@@ -178,4 +228,5 @@
             fake_sensor_commands="${fake_sensor_commands}"
             hand="${hand}"
+            ee_type="${ee_type}"
             bimanual="false"
             can_fd="${can_fd}"/>
@@ -200,4 +251,23 @@
         </xacro:if>
         </xacro:if>
+        <xacro:if value="${hand and ee_type == 'amazing_hand'}">
+        <xacro:property name="special_connection" value="$(arg special_connection)" />
+        <xacro:property name="connection" value="${special_connection if special_connection != '' else 'openarm' + '_link7'}" />
+        <xacro:amazing_hand_right
+            connected_to="${arm_prefix_modified}${connection}"
+            prefix="${arm_prefix_modified}ahand_"
+            xyz="$(arg xyz_ee)"
+            rpy="$(arg rpy_ee)"
+        />
+        <xacro:if value="${ros2_control}">
+            <xacro:include filename="$(find openarm_description)/urdf/ee/amazing_hand/ahand.ros2_control.xacro" />
+            <xacro:amazing_hand_ros2_control
+                prefix="${arm_prefix_modified}"
+                link_prefix="${arm_prefix_modified}ahand_"
+                joint_commands_topic="/ahand/joint_commands"
+                joint_states_topic="/ahand/joint_states"
+            />
+        </xacro:if>
+        </xacro:if>
         </xacro:if>
   </xacro:macro>

File: Open_arm_a1_ws/src/openarm_description/urdf/ros2_control/openarm.bimanual.ros2_control.xacro (robot description, xacro)
@@ -10,4 +10,5 @@
              fake_sensor_commands:=^|false
              hand:=^|false
+             ee_type:=^|openarm_hand
              left_arm_prefix:=^|left_
              right_arm_prefix:=^|right_
@@ -81,5 +82,5 @@
     </ros2_control>
     <!-- LEFT GRIPPER -->
-    <xacro:if value="${hand}">
+    <xacro:if value="${hand and ee_type == 'openarm_hand'}">
       <ros2_control name="openarm_left_gripper_hardware_interface" type="system">
         <hardware>
@@ -161,5 +162,5 @@
     </ros2_control>
     <!-- RIGHT GRIPPER -->
-    <xacro:if value="${hand}">
+    <xacro:if value="${hand and ee_type == 'openarm_hand'}">
       <ros2_control name="openarm_right_gripper_hardware_interface" type="system">
         <hardware>

File: Open_arm_a1_ws/src/openarm_description/urdf/ros2_control/openarm.ros2_control.xacro (robot description, xacro)
@@ -8,4 +8,5 @@
              fake_sensor_commands:=^|false
              hand:=^|false
+             ee_type:=^|openarm_hand
              gazebo_effort:=^|false
              arm_prefix:=''
@@ -71,5 +72,5 @@
       <xacro:configure_joint joint_name="openarm_${arm_prefix}joint6" initial_position="0.0"/>
       <xacro:configure_joint joint_name="openarm_${arm_prefix}joint7" initial_position="0.0"/>
-      <xacro:if value="${hand}">
+      <xacro:if value="${hand and ee_type == 'openarm_hand'}">
         <xacro:configure_joint joint_name="openarm_${arm_prefix}finger_joint1" initial_position="0.0" />
       </xacro:if>

Commit message: Refactor waypoint_recorder and remove unused components
- Removed the shellQuote function from waypoint_recorder.hpp and waypoint_recorder.cpp as it was no longer needed.
- Cleaned up record_waypoint_cli.cpp by eliminating the --auto-convert and --bt-out options, along with related logic.
- Deleted sequence_converter.h and sequence_converter.cpp files, which were not utilized in the current codebase.
- Updated CMakeLists.txt to remove references to the deleted sequence_converter source files.
- Added inertial properties to the openarm_robot.xacro file for the amazing_hand to improve gravity compensation.
- Removed the BehaviorTree.ROS2 submodule as it is no longer required.

File: Open_arm_a1_ws/src/openarm_description/urdf/robot/openarm_robot.xacro (robot description, xacro)
@@ -206,4 +206,35 @@
                         </geometry>
                     </collision>
+                    <!-- Lumped mass for the WHOLE amazing_hand, calibrated via
+                         gravity_calibration_tool (control/gravity_compensation_controller)
+                         against 6 real captured poses on real hardware: weighted
+                         least-squares fit against measured joint torque gave
+                         0.5938 kg, closely matching the hand's real measured
+                         weight (~0.5 kg) - validates that this connector (on the
+                         KDL chain, unlike most of the hand's own links which sit
+                         on branches invisible to chain-based gravity torque) is a
+                         sound place to lump it. Re-run the calibration tool if the
+                         connector's mount position or the real hand's mass changes. -->
+                         placed here for gravity_compensation_controller: the hand's
+                         own URDF is a closed-loop mechanism cut into an open tree,
+                         so most of its real link masses live on branches that
+                         aren't on the arm's base->hand_tcp KDL chain and are
+                         invisible to ChainDynParam-based static gravity torque no
+                         matter how accurate their individual values are. This
+                         connector link IS on that chain, has real mount geometry
+                         (unlike the zero-geometry ahand_root/hand_tcp reference
+                         links), and sits closest to the hand's actual mass - a
+                         reasonable single point to lump the whole hand's weight
+                         for gravity comp purposes. Origin/inertia are rough
+                         estimates (offset matches the visual mesh's own origin),
+                         not calibrated CAD values - fine for static gravity
+                         torque (mass + COM matter far more than the inertia
+                         tensor there), not precise enough for anything dynamic. -->
+                    <inertial>
+                        <origin xyz="0 0 -0.05" rpy="0 0 0" />
+                        <mass value="0.5938" />
+                        <inertia ixx="0.0006" ixy="0.0" ixz="0.0"
+                                 iyy="0.0006" iyz="0.0" izz="0.0004" />
+                    </inertial>
                 </link>
                 <joint name="openarm_${side}_ahand_connector_joint" type="fixed">
