Commit message: Add full Doxygen documentation for Open_arm_a1_ws
Adds \brief docs to every class, method, and free function across
openarm_description, communication, control, utilities, and builds
(openarm_description/scripts through builds/qvic_2026), plus a
Doxyfile and doc/groups.dox Topics page (Control/Communication/
Utilities/Description/Builds) so the generated docs guide by package
instead of showing a flat class list.

Co-Authored-By: Claude Sonnet 5 <noreply@anthropic.com>

File: Open_arm_a1_ws/src/openarm_description/urdf/robot/openarm_robot.xacro (robot description, xacro)
@@ -22,4 +22,6 @@
             can_interface:=''
             use_fake_hardware:=false
+            left_use_fake_hardware:='inherit'
+            right_use_fake_hardware:='inherit'
             head_use_fake_hardware:=false
             fake_sensor_commands:=false
@@ -141,4 +143,6 @@
             right_can_interface="${right_can_interface}"
             use_fake_hardware="${use_fake_hardware}"
+            left_use_fake_hardware="${left_use_fake_hardware}"
+            right_use_fake_hardware="${right_use_fake_hardware}"
             head_use_fake_hardware="${head_use_fake_hardware}"
             fake_sensor_commands="${fake_sensor_commands}"

File: Open_arm_a1_ws/src/openarm_description/urdf/robot/v10.urdf.xacro (robot description, xacro)
@@ -21,4 +21,6 @@
   <xacro:arg name="right_arm_prefix" default="right_" />
   <xacro:arg name="use_fake_hardware" default="false" />
+  <xacro:arg name="left_use_fake_hardware" default="inherit" />
+  <xacro:arg name="right_use_fake_hardware" default="inherit" />
   <xacro:arg name="head_use_fake_hardware" default="false" />
   <xacro:arg name="fake_sensor_commands" default="false" />
@@ -65,4 +67,6 @@
   right_arm_prefix="$(arg right_arm_prefix)"
   use_fake_hardware="$(arg use_fake_hardware)"
+  left_use_fake_hardware="$(arg left_use_fake_hardware)"
+  right_use_fake_hardware="$(arg right_use_fake_hardware)"
   head_use_fake_hardware="$(arg head_use_fake_hardware)"
   fake_sensor_commands="$(arg fake_sensor_commands)"

File: Open_arm_a1_ws/src/openarm_description/urdf/ros2_control/openarm.bimanual.ros2_control.xacro (robot description, xacro)
@@ -7,4 +7,6 @@
              right_can_interface:=^|can0
              use_fake_hardware:=^|false
+             left_use_fake_hardware:=^|inherit
+             right_use_fake_hardware:=^|inherit
              head_use_fake_hardware:=^|false
              fake_sensor_commands:=^|false
@@ -25,4 +27,12 @@
              no_prefix:=^|false">
     <xacro:property name="body_joint_prefix" value="${'' if no_prefix else 'openarm_body_'}" />
+    <!-- left_use_fake_hardware/right_use_fake_hardware:='inherit' (default) falls
+         back to the shared use_fake_hardware, so callers that only know about
+         use_fake_hardware (sequence_executor.launch.py, robot_api.launch.py, etc.)
+         keep their existing all-or-nothing behavior unchanged. Pass an explicit
+         'true'/'false' per side to override just that arm - see bringup.launch.py's
+         left_arm/right_arm launch args. -->
+    <xacro:property name="left_fake_hw" value="${use_fake_hardware if left_use_fake_hardware == 'inherit' else left_use_fake_hardware}" />
+    <xacro:property name="right_fake_hw" value="${use_fake_hardware if right_use_fake_hardware == 'inherit' else right_use_fake_hardware}" />
     <xacro:macro name="configure_arm_joint" params="joint_name initial_position">
       <joint name="${joint_name}">
@@ -44,10 +54,10 @@
         <hardware>
           <param name="arm_type">${arm_type}</param>
-          <xacro:if value="${use_fake_hardware}">
-            <plugin>mock_components/GenericSystem</plugin>
-            <param name="fake_sensor_commands">${fake_sensor_commands}</param>
-            <param name="state_following_offset">0.0</param>
-          </xacro:if>
-          <xacro:unless value="${use_fake_hardware}">
+          <xacro:if value="${left_fake_hw}">
+            <plugin>mock_components/GenericSystem</plugin>
+            <param name="fake_sensor_commands">${fake_sensor_commands}</param>
+            <param name="state_following_offset">0.0</param>
+          </xacro:if>
+          <xacro:unless value="${left_fake_hw}">
             <xacro:if value="${gazebo}">
               <plugin>gz_ros2_control/GazeboSimSystem</plugin>
@@ -102,10 +112,10 @@
       <ros2_control name="openarm_left_gripper_hardware_interface" type="system">
         <hardware>
-          <xacro:if value="${use_fake_hardware}">
-            <plugin>mock_components/GenericSystem</plugin>
-            <param name="fake_sensor_commands">${fake_sensor_commands}</param>
-            <param name="state_following_offset">0.0</param>
-          </xacro:if>
-          <xacro:unless value="${use_fake_hardware}">
+          <xacro:if value="${left_fake_hw}">
+            <plugin>mock_components/GenericSystem</plugin>
+            <param name="fake_sensor_commands">${fake_sensor_commands}</param>
+            <param name="state_following_offset">0.0</param>
+          </xacro:if>
+          <xacro:unless value="${left_fake_hw}">
             <xacro:if value="${gazebo}">
               <plugin>gz_ros2_control/GazeboSimSystem</plugin>
@@ -121,5 +131,5 @@
              fake/gazebo path - declaring it in both components crashes
              controller_manager with a duplicate CommandInterface key. -->
-        <xacro:if value="${use_fake_hardware or gazebo}">
+        <xacro:if value="${left_fake_hw or gazebo}">
           <xacro:configure_arm_joint joint_name="openarm_${left_arm_prefix}finger_joint1" initial_position="0.0" />
         </xacro:if>
@@ -139,13 +149,13 @@
          (JointTrajectoryController goals get rejected with no reason
          logged). -->
-    <xacro:if value="${hand and ee_type == 'amazing_hand' and (use_fake_hardware or gazebo)}">
+    <xacro:if value="${hand and ee_type == 'amazing_hand' and (left_fake_hw or gazebo)}">
       <ros2_control name="openarm_left_hand_rotate_hardware_interface" type="system">
         <hardware>
-          <xacro:if value="${use_fake_hardware}">
-            <plugin>mock_components/GenericSystem</plugin>
-            <param name="fake_sensor_commands">${fake_sensor_commands}</param>
-            <param name="state_following_offset">0.0</param>
-          </xacro:if>
-          <xacro:unless value="${use_fake_hardware}">
+          <xacro:if value="${left_fake_hw}">
+            <plugin>mock_components/GenericSystem</plugin>
+            <param name="fake_sensor_commands">${fake_sensor_commands}</param>
+            <param name="state_following_offset">0.0</param>
+          </xacro:if>
+          <xacro:unless value="${left_fake_hw}">
             <plugin>gz_ros2_control/GazeboSimSystem</plugin>
           </xacro:unless>
@@ -157,10 +167,10 @@
         <hardware>
           <param name="arm_type">${arm_type}</param>
-          <xacro:if value="${use_fake_hardware}">
-            <plugin>mock_components/GenericSystem</plugin>
-            <param name="fake_sensor_commands">${fake_sensor_commands}</param>
-            <param name="state_following_offset">0.0</param>
-          </xacro:if>
-          <xacro:unless value="${use_fake_hardware}">
+          <xacro:if value="${right_fake_hw}">
+            <plugin>mock_components/GenericSystem</plugin>
+            <param name="fake_sensor_commands">${fake_sensor_commands}</param>
+            <param name="state_following_offset">0.0</param>
+          </xacro:if>
+          <xacro:unless value="${right_fake_hw}">
             <xacro:if value="${gazebo}">
               <plugin>gz_ros2_control/GazeboSimSystem</plugin>
@@ -210,10 +220,10 @@
       <ros2_control name="openarm_right_gripper_hardware_interface" type="system">
         <hardware>
-          <xacro:if value="${use_fake_hardware}">
-            <plugin>mock_components/GenericSystem</plugin>
-            <param name="fake_sensor_commands">${fake_sensor_commands}</param>
-            <param name="state_following_offset">0.0</param>
-          </xacro:if>
-          <xacro:unless value="${use_fake_hardware}">
+          <xacro:if value="${right_fake_hw}">
+            <plugin>mock_components/GenericSystem</plugin>
+            <param name="fake_sensor_commands">${fake_sensor_commands}</param>
+            <param name="state_following_offset">0.0</param>
+          </xacro:if>
+          <xacro:unless value="${right_fake_hw}">
             <xacro:if value="${gazebo}">
               <plugin>gz_ros2_control/GazeboSimSystem</plugin>
@@ -229,5 +239,5 @@
              fake/gazebo path - declaring it in both components crashes
              controller_manager with a duplicate CommandInterface key. -->
-        <xacro:if value="${use_fake_hardware or gazebo}">
+        <xacro:if value="${right_fake_hw or gazebo}">
           <xacro:configure_arm_joint joint_name="openarm_${right_arm_prefix}finger_joint1" initial_position="0.0" />
         </xacro:if>
@@ -237,13 +247,13 @@
     <!-- RIGHT "MOTOR 8" - see openarm_left_hand_rotate_hardware_interface's
          comment above. -->
-    <xacro:if value="${hand and ee_type == 'amazing_hand' and (use_fake_hardware or gazebo)}">
+    <xacro:if value="${hand and ee_type == 'amazing_hand' and (right_fake_hw or gazebo)}">
       <ros2_control name="openarm_right_hand_rotate_hardware_interface" type="system">
         <hardware>
-          <xacro:if value="${use_fake_hardware}">
-            <plugin>mock_components/GenericSystem</plugin>
-            <param name="fake_sensor_commands">${fake_sensor_commands}</param>
-            <param name="state_following_offset">0.0</param>
-          </xacro:if>
-          <xacro:unless value="${use_fake_hardware}">
+          <xacro:if value="${right_fake_hw}">
+            <plugin>mock_components/GenericSystem</plugin>
+            <param name="fake_sensor_commands">${fake_sensor_commands}</param>
+            <param name="state_following_offset">0.0</param>
+          </xacro:if>
+          <xacro:unless value="${right_fake_hw}">
             <plugin>gz_ros2_control/GazeboSimSystem</plugin>
           </xacro:unless>
