Commit message: refactor: update BehaviorTree.ROS2 architecture and improve URDF robot descriptions

File: Open_arm_a1_ws/src/openarm_description/urdf/base/openarm_base.xacro (robot description, xacro)
@@ -95,5 +95,5 @@
       <parent link="${prefix}link" />
       <child link="${prefix}left_drive_wheel_link" />
-      <axis xyz="0 0.000125537276710988 -0.999999992120196" />
+      <axis xyz="0 0.000125537276710988 0.999999992120196" />
     </joint>
     <xacro:base_caster prefix="${prefix}" description_pkg="${description_pkg}" corner="fr"
@@ -109,4 +109,19 @@
                        caster_xyz="-0.152199376082463 0.0939770926972477 -0.2186"
                        wheel_z="5.79435111003335E-12" />
+    <!-- Gazebo: drive wheels có ma sát cao để bám đường -->
+    <gazebo reference="${prefix}right_drive_wheel_link">
+      <mu1>1.5</mu1>
+      <mu2>1.5</mu2>
+      <kp>1000000.0</kp>
+      <kd>100.0</kd>
+      <minDepth>0.001</minDepth>
+    </gazebo>
+    <gazebo reference="${prefix}left_drive_wheel_link">
+      <mu1>1.5</mu1>
+      <mu2>1.5</mu2>
+      <kp>1000000.0</kp>
+      <kd>100.0</kd>
+      <minDepth>0.001</minDepth>
+    </gazebo>
   </xacro:macro>
 </robot>

File: Open_arm_a1_ws/src/openarm_description/urdf/base/openarm_base_macro.xacro (robot description, xacro)
@@ -29,4 +29,5 @@
       <child link="${prefix}${corner}_caster_link" />
       <axis xyz="0 0 1" />
+      <dynamics damping="0.01" friction="0.0"/>
     </joint>
     <link name="${prefix}${corner}_wheel_link">
@@ -56,5 +57,14 @@
       <child link="${prefix}${corner}_wheel_link" />
       <axis xyz="0 0 1" />
+      <dynamics damping="0.005" friction="0.0"/>
     </joint>
+    <!-- Gazebo: caster wheel có ma sát thấp để trượt dễ dàng -->
+    <gazebo reference="${prefix}${corner}_wheel_link">
+      <mu1>0.1</mu1>
+      <mu2>0.1</mu2>
+      <kp>1000000.0</kp>
+      <kd>100.0</kd>
+      <minDepth>0.001</minDepth>
+    </gazebo>
   </xacro:macro>
 </robot>

File: Open_arm_a1_ws/src/openarm_description/urdf/ee/openarm_hand.xacro (robot description, xacro)
@@ -68,5 +68,6 @@
       <axis xyz="0 1 0" />
       <limit effort="333" lower="0.0" upper="0.044" velocity="10.0" />
-      <mimic joint="${ee_prefix}finger_joint1" />
+      <!-- mimic removed: DART physics in Gazebo Sim does not support mimic constraints.
+           finger_joint2 is controlled directly via ros2_control gripper controller instead. -->
     </joint>
   </xacro:macro>

File: Open_arm_a1_ws/src/openarm_description/urdf/robot/openarm_robot.xacro (robot description, xacro)
@@ -39,4 +39,5 @@
             right_arm_prefix:='right_'
             can_fd:='true'
+            gazebo:=false
             mobile_base:=false
             mobile_base_xyz:='0 0 0'
@@ -66,5 +67,5 @@
         <xacro:openarm_base
         description_pkg="openarm_description"
-        connected_to="${body_connected_to}"
+        connected_to=""
         xyz="${mobile_base_xyz}"
         rpy="${mobile_base_rpy}" />
@@ -123,4 +124,5 @@
             left_arm_prefix="${left_arm_prefix}"
             right_arm_prefix="${right_arm_prefix}"
+            gazebo="${gazebo}"
             hand="${hand}"/>
         </xacro:if>

File: Open_arm_a1_ws/src/openarm_description/urdf/robot/v10.urdf (robot description, URDF)
Before this commit: robot openarm, 37 links, 36 joints
Joints:
- joint openarm_base_right_drive_wheel_joint: axis 0 0.000125537276711018 0.999999992120196 -> 0 0 1; origin xyz=-0.00217824370780602 -0.218924944717817 -0.224330452201286 rpy=-1.5707963267949 0 0 -> xyz=-0.00217824370780602 -0.218924944717817 -0.224330452201286 rpy=1.5707963267949 0 0

File: Open_arm_a1_ws/src/openarm_description/urdf/robot/v10.urdf.xacro (robot description, xacro)
@@ -28,4 +28,5 @@
   <xacro:arg name="left_arm_base_rpy" default="-1.5708 0 3.14159" />
   <xacro:arg name="can_fd" default="true" />
+  <xacro:arg name="gazebo" default="false" />
   <xacro:arg name="mobile_base" default="false" />
   <xacro:arg name="mobile_base_xyz" default="0 0 0.31" />
@@ -70,4 +71,5 @@
   left_arm_base_rpy="$(arg left_arm_base_rpy)"
   can_fd="$(arg can_fd)"
+  gazebo="$(arg gazebo)"
   mobile_base="$(arg mobile_base)"
   mobile_base_xyz="$(arg mobile_base_xyz)"

File: Open_arm_a1_ws/src/openarm_description/urdf/ros2_control/openarm.bimanual.ros2_control.xacro (robot description, xacro)
@@ -12,6 +12,22 @@
              left_arm_prefix:=^|left_
              right_arm_prefix:=^|right_
+             gazebo:=^|false
              can_fd:=^|true">
-    <!-- Left Arm Hardware Interface -->
+    <xacro:macro name="configure_arm_joint" params="joint_name initial_position">
+      <joint name="${joint_name}">
+        <command_interface name="position"/>
+        <command_interface name="velocity"/>
+        <command_interface name="effort"/>
+        <state_interface name="position">
+          <param name="initial_value">${initial_position}</param>
+        </state_interface>
+        <state_interface name="velocity">
+          <param name="initial_value">0.0</param>
+        </state_interface>
+        <state_interface name="effort">
+          <param name="initial_value">0.0</param>
+        </state_interface>
+      </joint>
+    </xacro:macro>
     <ros2_control name="openarm_left_hardware_interface" type="system">
         <hardware>
@@ -49,29 +65,43 @@
               <param name="kd7">${control_gains['joint7']['kd']}</param>
             </xacro:unless>
+          <xacro:if value="${use_fake_hardware}">
+            <plugin>mock_components/GenericSystem</plugin>
+            <param name="fake_sensor_commands">${fake_sensor_commands}</param>
+            <param name="state_following_offset">0.0</param>
+          </xacro:if>
+          <xacro:unless value="${use_fake_hardware}">
+            <xacro:if value="${gazebo}">
+              <plugin>gz_ros2_control/GazeboSimSystem</plugin>
+            </xacro:if>
+            <xacro:unless value="${gazebo}">
+              <plugin>openarm_hardware/OpenArm_v10HW</plugin>
+              <param name="can_interface">${left_can_interface}</param>
+              <param name="arm_prefix">${left_arm_prefix}</param>
+              <param name="hand">${hand}</param>
+              <param name="can_fd">${can_fd}</param>
+              <param name="kp1">${control_gains['joint1']['kp']}</param>
+              <param name="kp2">${control_gains['joint2']['kp']}</param>
+              <param name="kp3">${control_gains['joint3']['kp']}</param>
+              <param name="kp4">${control_gains['joint4']['kp']}</param>
+              <param name="kp5">${control_gains['joint5']['kp']}</param>
+              <param name="kp6">${control_gains['joint6']['kp']}</param>
+              <param name="kp7">${control_gains['joint7']['kp']}</param>
+              <param name="kd1">${control_gains['joint1']['kd']}</param>
+              <param name="kd2">${control_gains['joint2']['kd']}</param>
+              <param name="kd3">${control_gains['joint3']['kd']}</param>
+              <param name="kd4">${control_gains['joint4']['kd']}</param>
+              <param name="kd5">${control_gains['joint5']['kd']}</param>
+              <param name="kd6">${control_gains['joint6']['kd']}</param>
+              <param name="kd7">${control_gains['joint7']['kd']}</param>
+            </xacro:unless>
           </xacro:unless>
         </hardware>
-      <xacro:macro name="configure_joint" params="joint_name initial_position">
-        <joint name="${joint_name}">
-          <command_interface name="position"/>
-          <command_interface name="velocity"/>
-          <command_interface name="effort"/>
-          <state_interface name="position">
-            <param name="initial_value">${initial_position}</param>
-          </state_interface>
-          <state_interface name="velocity">
-            <param name="initial_value">0.0</param>
-          </state_interface>
-          <state_interface name="effort">
-            <param name="initial_value">0.0</param>
-          </state_interface>
-        </joint>
-      </xacro:macro>
-      <xacro:configure_joint joint_name="openarm_${left_arm_prefix}joint1" initial_position="0.0"/>
-      <xacro:configure_joint joint_name="openarm_${left_arm_prefix}joint2" initial_position="0.0"/>
-      <xacro:configure_joint joint_name="openarm_${left_arm_prefix}joint3" initial_position="0.0"/>
-      <xacro:configure_joint joint_name="openarm_${left_arm_prefix}joint4" initial_position="0.0"/>
-      <xacro:configure_joint joint_name="openarm_${left_arm_prefix}joint5" initial_position="0.0"/>
-      <xacro:configure_joint joint_name="openarm_${left_arm_prefix}joint6" initial_position="0.0"/>
-      <xacro:configure_joint joint_name="openarm_${left_arm_prefix}joint7" initial_position="0.0"/>
+      <xacro:configure_arm_joint joint_name="openarm_${left_arm_prefix}joint1" initial_position="0.0"/>
+      <xacro:configure_arm_joint joint_name="openarm_${left_arm_prefix}joint2" initial_position="0.0"/>
+      <xacro:configure_arm_joint joint_name="openarm_${left_arm_prefix}joint3" initial_position="0.0"/>
+      <xacro:configure_arm_joint joint_name="openarm_${left_arm_prefix}joint4" initial_position="0.0"/>
+      <xacro:configure_arm_joint joint_name="openarm_${left_arm_prefix}joint5" initial_position="0.0"/>
+      <xacro:configure_arm_joint joint_name="openarm_${left_arm_prefix}joint6" initial_position="0.0"/>
+      <xacro:configure_arm_joint joint_name="openarm_${left_arm_prefix}joint7" initial_position="0.0"/>
       <xacro:if value="${hand}">
         <xacro:configure_joint joint_name="openarm_${left_arm_prefix}finger_joint1" initial_position="0.0" />
@@ -91,7 +121,8 @@
           </joint>
         </xacro:if>
+        <xacro:configure_arm_joint joint_name="openarm_${left_arm_prefix}finger_joint1" initial_position="0.0" />
+        <xacro:configure_arm_joint joint_name="openarm_${left_arm_prefix}finger_joint2" initial_position="0.0" />
       </xacro:if>
     </ros2_control>
-    <!-- Right Arm Hardware Interface -->
     <ros2_control name="openarm_right_hardware_interface" type="system">
         <hardware>
@@ -129,13 +160,43 @@
               <param name="kd7">${control_gains['joint7']['kd']}</param>
             </xacro:unless>
+          <xacro:if value="${use_fake_hardware}">
+            <plugin>mock_components/GenericSystem</plugin>
+            <param name="fake_sensor_commands">${fake_sensor_commands}</param>
+            <param name="state_following_offset">0.0</param>
+          </xacro:if>
+          <xacro:unless value="${use_fake_hardware}">
+            <xacro:if value="${gazebo}">
+              <plugin>gz_ros2_control/GazeboSimSystem</plugin>
+            </xacro:if>
+            <xacro:unless value="${gazebo}">
+              <plugin>openarm_hardware/OpenArm_v10HW</plugin>
+              <param name="can_interface">${right_can_interface}</param>
+              <param name="arm_prefix">${right_arm_prefix}</param>
+              <param name="hand">${hand}</param>
+              <param name="can_fd">${can_fd}</param>
+              <param name="kp1">${control_gains['joint1']['kp']}</param>
+              <param name="kp2">${control_gains['joint2']['kp']}</param>
+              <param name="kp3">${control_gains['joint3']['kp']}</param>
+              <param name="kp4">${control_gains['joint4']['kp']}</param>
+              <param name="kp5">${control_gains['joint5']['kp']}</param>
+              <param name="kp6">${control_gains['joint6']['kp']}</param>
+              <param name="kp7">${control_gains['joint7']['kp']}</param>
+              <param name="kd1">${control_gains['joint1']['kd']}</param>
+              <param name="kd2">${control_gains['joint2']['kd']}</param>
+              <param name="kd3">${control_gains['joint3']['kd']}</param>
+              <param name="kd4">${control_gains['joint4']['kd']}</param>
+              <param name="kd5">${control_gains['joint5']['kd']}</param>
+              <param name="kd6">${control_gains['joint6']['kd']}</param>
+              <param name="kd7">${control_gains['joint7']['kd']}</param>
+            </xacro:unless>
           </xacro:unless>
         </hardware>
-      <xacro:configure_joint joint_name="openarm_${right_arm_prefix}joint1" initial_position="0.0"/>
-      <xacro:configure_joint joint_name="openarm_${right_arm_prefix}joint2" initial_position="0.0"/>
-      <xacro:configure_joint joint_name="openarm_${right_arm_prefix}joint3" initial_position="0.0"/>
-      <xacro:configure_joint joint_name="openarm_${right_arm_prefix}joint4" initial_position="0.0"/>
-      <xacro:configure_joint joint_name="openarm_${right_arm_prefix}joint5" initial_position="0.0"/>
-      <xacro:configure_joint joint_name="openarm_${right_arm_prefix}joint6" initial_position="0.0"/>
-      <xacro:configure_joint joint_name="openarm_${right_arm_prefix}joint7" initial_position="0.0"/>
+      <xacro:configure_arm_joint joint_name="openarm_${right_arm_prefix}joint1" initial_position="0.0"/>
+      <xacro:configure_arm_joint joint_name="openarm_${right_arm_prefix}joint2" initial_position="0.0"/>
+      <xacro:configure_arm_joint joint_name="openarm_${right_arm_prefix}joint3" initial_position="0.0"/>
+      <xacro:configure_arm_joint joint_name="openarm_${right_arm_prefix}joint4" initial_position="0.0"/>
+      <xacro:configure_arm_joint joint_name="openarm_${right_arm_prefix}joint5" initial_position="0.0"/>
+      <xacro:configure_arm_joint joint_name="openarm_${right_arm_prefix}joint6" initial_position="0.0"/>
+      <xacro:configure_arm_joint joint_name="openarm_${right_arm_prefix}joint7" initial_position="0.0"/>
       <xacro:if value="${hand}">
         <xacro:configure_joint joint_name="openarm_${right_arm_prefix}finger_joint1" initial_position="0.0" />
@@ -155,23 +216,48 @@
           </joint>
         </xacro:if>
+        <xacro:configure_arm_joint joint_name="openarm_${right_arm_prefix}finger_joint1" initial_position="0.0" />
+        <xacro:configure_arm_joint joint_name="openarm_${right_arm_prefix}finger_joint2" initial_position="0.0" />
       </xacro:if>
     </ros2_control>
-    <!-- Base Hardware Interface -->
     <ros2_control name="openarm_base_hardware_interface" type="system">
         <hardware>
-          <plugin>mock_components/GenericSystem</plugin>
-          <param name="state_following_offset">0.0</param>
+          <xacro:if value="${use_fake_hardware}">
+            <plugin>mock_components/GenericSystem</plugin>
+            <param name="calculate_dynamics">true</param>
+          </xacro:if>
+          <xacro:unless value="${use_fake_hardware}">
+            <xacro:if value="${gazebo}">
+              <plugin>gz_ros2_control/GazeboSimSystem</plugin>
+            </xacro:if>
+            <xacro:unless value="${gazebo}">
+              <!-- Ở thực tế, bạn có thể thay thế driver thật cho đế xe ở đây nếu có -->
+              <plugin>mock_components/GenericSystem</plugin>
+            </xacro:unless>
+          </xacro:unless>
         </hardware>
-      <xacro:configure_joint joint_name="openarm_base_fl_caster_joint" initial_position="0.0"/>
-      <xacro:configure_joint joint_name="openarm_base_fl_wheel_joint" initial_position="0.0"/>
-      <xacro:configure_joint joint_name="openarm_base_fr_caster_joint" initial_position="0.0"/>
-      <xacro:configure_joint joint_name="openarm_base_fr_wheel_joint" initial_position="0.0"/>
-      <xacro:configure_joint joint_name="openarm_base_bl_caster_joint" initial_position="0.0"/>
-      <xacro:configure_joint joint_name="openarm_base_bl_wheel_joint" initial_position="0.0"/>
-      <xacro:configure_joint joint_name="openarm_base_br_caster_joint" initial_position="0.0"/>
-      <xacro:configure_joint joint_name="openarm_base_br_wheel_joint" initial_position="0.0"/>
-      <xacro:configure_joint joint_name="openarm_base_left_drive_wheel_joint" initial_position="0.0"/>
-      <xacro:configure_joint joint_name="openarm_base_right_drive_wheel_joint" initial_position="0.0"/>
+        <joint name="openarm_base_left_drive_wheel_joint">
+            <command_interface name="velocity"/>
+            <state_interface name="velocity"/>
+            <state_interface name="position"/>
+        </joint>
+        <joint name="openarm_base_right_drive_wheel_joint">
+            <command_interface name="velocity"/>
+            <state_interface name="velocity"/>
+            <state_interface name="position"/>
+        </joint>
+        <joint name="openarm_base_fl_caster_joint"><state_interface name="position"><param name="initial_value">0.0</param></state_interface></joint>
+        <joint name="openarm_base_fr_caster_joint"><state_interface name="position"><param name="initial_value">0.0</param></state_interface></joint>
+        <joint name="openarm_base_bl_caster_joint"><state_interface name="position"><param name="initial_value">0.0</param></state_interface></joint>
+        <joint name="openarm_base_br_caster_joint"><state_interface name="position"><param name="initial_value">0.0</param></state_interface></joint>
+        <joint name="openarm_base_fl_wheel_joint"><state_interface name="position"><param name="initial_value">0.0</param></state_interface></joint>
+        <joint name="openarm_base_fr_wheel_joint"><state_interface name="position"><param name="initial_value">0.0</param></state_interface></joint>
+        <joint name="openarm_base_bl_wheel_joint"><state_interface name="position"><param name="initial_value">0.0</param></state_interface></joint>
+        <joint name="openarm_base_br_wheel_joint"><state_interface name="position"><param name="initial_value">0.0</param></state_interface></joint>
     </ros2_control>
   </xacro:macro>
+  <gazebo>
+    <plugin name="gz_ros2_control::GazeboSimROS2ControlPlugin" filename="libgz_ros2_control-system.so">
+      <parameters>$(find arm_control)/config/bimanual_controllers.yaml</parameters>
+    </plugin>
+  </gazebo>
 </robot>
