Commit message: feat: add body v2 articulated neck and head support with joint limits and controllers

File: Open_arm_a1_ws/src/openarm_description/urdf/base/openarm_base.xacro (robot description, xacro)
@@ -22,5 +22,20 @@
       </joint>
     </xacro:if>
-    <link name="${prefix}link">
+    <!-- "${prefix}link" (the externally-visible root name; SRDF's virtual_joint and
+         everything else that names "openarm_base_link" targets this) is kept as an
+         empty anchor, not the mesh/wheels holder. The mesh's own origin sits at
+         wheel-axle height (the drive/caster wheel joints are ~0.22-0.27m below it),
+         not at the ground; with no localization publishing a real world transform,
+         that made the whole base render sunk into the floor. This fixed joint
+         re-grounds it: floor at this link's origin, mesh+wheels (unchanged,
+         untouched below) hang appropriately below/around it, matching where the
+         wheels actually reach the ground. -->
+    <link name="${prefix}link" />
+    <joint name="${prefix}floor_offset_joint" type="fixed">
+      <parent link="${prefix}link" />
+      <child link="${prefix}link_body" />
+      <origin xyz="0 0 0.31" rpy="0 0 0" />
+    </joint>
+    <link name="${prefix}link_body">
       <inertial>
         <origin xyz="0.0139877464492624 -5.68244441146032E-05 -0.124578208571542" rpy="0 0 0" />
@@ -66,5 +81,5 @@
     <joint name="${prefix}right_drive_wheel_joint" type="continuous">
       <origin xyz="-0.00217824370780602 -0.218924944717817 -0.224330452201286" rpy="-1.5707963267949 0 0" />
-      <parent link="${prefix}link" />
+      <parent link="${prefix}link_body" />
       <child link="${prefix}right_drive_wheel_link" />
       <axis xyz="0 0.000125537276711018 0.999999992120196" />
@@ -93,5 +108,5 @@
     <joint name="${prefix}left_drive_wheel_joint" type="continuous">
       <origin xyz="-0.00217793050105813 0.218879130112312 -0.224330452201204" rpy="-1.5707963267949 0 0" />
-      <parent link="${prefix}link" />
+      <parent link="${prefix}link_body" />
       <child link="${prefix}left_drive_wheel_link" />
       <axis xyz="0 0.000125537276710988 0.999999992120196" />
@@ -99,14 +114,14 @@
     <xacro:base_caster prefix="${prefix}" description_pkg="${description_pkg}" corner="fr"
                        caster_xyz="0.149800623917563 -0.0925229073028034 -0.2186"
-                       wheel_z="-0.00149999999415462" />
+                       wheel_z="-0.00149999999415462" parent_link="${prefix}link_body" />
     <xacro:base_caster prefix="${prefix}" description_pkg="${description_pkg}" corner="fl"
                        caster_xyz="0.149800623917537 0.0924770926972476 -0.2186"
-                       wheel_z="0.00150000000579448" />
+                       wheel_z="0.00150000000579448" parent_link="${prefix}link_body" />
     <xacro:base_caster prefix="${prefix}" description_pkg="${description_pkg}" corner="br"
                        caster_xyz="-0.152199376082463 -0.0940229073027524 -0.2186"
-                       wheel_z="5.79430947666992E-12" />
+                       wheel_z="5.79430947666992E-12" parent_link="${prefix}link_body" />
     <xacro:base_caster prefix="${prefix}" description_pkg="${description_pkg}" corner="bl"
                        caster_xyz="-0.152199376082463 0.0939770926972477 -0.2186"
-                       wheel_z="5.79435111003335E-12" />
+                       wheel_z="5.79435111003335E-12" parent_link="${prefix}link_body" />
     <!-- Gazebo: drive wheels có ma sát cao để bám đường -->
     <gazebo reference="${prefix}right_drive_wheel_link">

File: Open_arm_a1_ws/src/openarm_description/urdf/base/openarm_base_macro.xacro (robot description, xacro)
@@ -2,5 +2,5 @@
 <robot xmlns:xacro="http://www.ros.org/wiki/xacro">
   <xacro:macro name="base_caster"
-               params="prefix description_pkg corner caster_xyz wheel_z">
+               params="prefix description_pkg corner caster_xyz wheel_z parent_link:='${prefix}link'">
     <link name="${prefix}${corner}_caster_link">
       <inertial>
@@ -26,5 +26,5 @@
     <joint name="${prefix}${corner}_caster_joint" type="continuous">
       <origin xyz="${caster_xyz}" rpy="0 0 0" />
-      <parent link="${prefix}link" />
+      <parent link="${parent_link}" />
       <child link="${prefix}${corner}_caster_link" />
       <axis xyz="0 0 1" />

File: Open_arm_a1_ws/src/openarm_description/urdf/body/openarm_body.xacro (robot description, xacro)
@@ -25,11 +25,18 @@
       </joint>
     </xacro:if>
-    <!-- v2's chassis mesh (chasssis_link.STL, base-plate component stripped out) is
-         already centered on its mount point, already in meters, and carries its own
-         correctly-measured inertial; v1/v10's raw mesh is in mm and isn't centered,
-         so they need the baked-in offset + scale instead. -->
     <xacro:property name="mesh_xyz" value="${'0 0 0' if body_type == 'v2' else '-0.251 0.1302 -0.210104'}" />
     <xacro:property name="mesh_rpy" value="${'0 0 0' if body_type == 'v2' else '0 0 -1.5708'}" />
     <xacro:property name="mesh_scale" value="${'1 1 1' if body_type == 'v2' else '0.001 0.001 0.001'}" />
+    <xacro:property name="neck_mesh_xyz" value="0 0 0" />
+    <xacro:property name="neck_mesh_rpy" value="0 0 0" />
+    <xacro:property name="head_mesh_xyz" value="0 0 0" />
+    <xacro:property name="head_mesh_rpy" value="0 0 0" />
+    <!-- Outer cosmetic shell cover (RobotShell.STL). Came as a loose file with no
+         URDF of its own, so there's no reference joint origin to copy like the
+         chassis/neck/head had - start at identity and nudge from here. Note it's
+         in millimeters unlike the other v2 meshes, hence the scale. -->
+    <xacro:property name="shell_mesh_xyz" value="0.12 0 -0.27" />
+    <xacro:property name="shell_mesh_rpy" value="0 0 -1.5707" />
+    <xacro:property name="shell_mesh_scale" value="0.001 0.001 0.001" />
     <link name="${prefix}link0">
       <visual>
@@ -69,5 +76,5 @@
       <link name="${prefix}neck_link">
         <visual>
-          <origin xyz="0 0 0" rpy="0 0 0" />
+          <origin xyz="${neck_mesh_xyz}" rpy="${neck_mesh_rpy}" />
           <geometry>
             <mesh filename="package://${description_pkg}/meshes/body/${body_type}/visual/Neck_Link.STL" />
@@ -75,5 +82,5 @@
         </visual>
         <collision>
-          <origin xyz="0 0 0" rpy="0 0 0" />
+          <origin xyz="${neck_mesh_xyz}" rpy="${neck_mesh_rpy}" />
           <geometry>
             <mesh filename="package://${description_pkg}/meshes/body/${body_type}/collision/Neck_Link_symp.STL" />
@@ -97,5 +104,5 @@
       <link name="${prefix}head_link">
         <visual>
-          <origin xyz="0 0 0" rpy="0 0 0" />
+          <origin xyz="${head_mesh_xyz}" rpy="${head_mesh_rpy}" />
           <geometry>
             <mesh filename="package://${description_pkg}/meshes/body/${body_type}/visual/Head_Link.STL" />
@@ -103,5 +110,5 @@
         </visual>
         <collision>
-          <origin xyz="0 0 0" rpy="0 0 0" />
+          <origin xyz="${head_mesh_xyz}" rpy="${head_mesh_rpy}" />
           <geometry>
             <mesh filename="package://${description_pkg}/meshes/body/${body_type}/collision/Head_Link_symp.STL" />
@@ -123,4 +130,18 @@
         <limit lower="-1.57" upper="1.57" effort="10" velocity="3" />
       </joint>
+      <!-- Cosmetic outer shell, visual-only (no collision geometry, doesn't
+           block planning) -->
+      <link name="${prefix}shell_link">
+        <visual>
+          <origin xyz="${shell_mesh_xyz}" rpy="${shell_mesh_rpy}" />
+          <geometry>
+            <mesh filename="package://${description_pkg}/meshes/body/${body_type}/visual/RobotShell.STL" scale="${shell_mesh_scale}" />
+          </geometry>
+        </visual>
+      </link>
+      <joint name="${prefix}shell_joint" type="fixed">
+        <parent link="${prefix}link0" />
+        <child link="${prefix}shell_link" />
+      </joint>
     </xacro:if>
   </xacro:macro>

File: Open_arm_a1_ws/src/openarm_description/urdf/robot/openarm_robot.xacro (robot description, xacro)
@@ -66,4 +66,12 @@
     <xacro:property name="body_prefix_modified" value="${'' if body_prefix == '' else body_prefix + '_'}" />
     <xacro:property name="base_link_name" value="openarm_base_link" />
+    <!-- Body mounts onto the base's mesh-bearing link, not the outer anchor:
+         openarm_base_link is an empty anchor sitting 0.31m below
+         openarm_base_link_body (see openarm_base.xacro's floor_offset_joint,
+         which lifts the mesh/wheels off the anchor so the base renders on
+         the floor instead of sunk into it). The body/torso needs to sit on
+         top of the actual base mesh, so it has to hang off that same lifted
+         link, not the un-lifted anchor underneath it. -->
+    <xacro:property name="base_mount_link_name" value="openarm_base_link_body" />
     <xacro:if value="${mobile_base}">
         <xacro:openarm_base
@@ -74,4 +82,9 @@
     </xacro:if>
     <xacro:if value="${bimanual}">
+        <!-- body_link0's own mesh origin sits mid-mesh (bottom extends 0.662m below
+             it, verified via STL bounding box), while the base mount link's origin
+             sits at its own mesh's top surface. Mounting at zero offset buries most
+             of the chassis inside/below the base, so v2 needs this extra lift on
+             top of whatever mobile_base_body_xyz the caller supplied. -->
         <xacro:openarm_body
         body_type="${body_type}"
@@ -79,7 +92,7 @@
         no_prefix="${no_prefix}"
         description_pkg="openarm_description"
-        connected_to="${base_link_name if mobile_base else body_connected_to}"
-        xyz="${mobile_base_body_xyz if mobile_base else xyz}"
-        rpy="${mobile_base_body_rpy if mobile_base else rpy}"
+        connected_to="${base_mount_link_name if mobile_base else body_connected_to}"
+        xyz="${('0.061 0.006 0.662' if body_type == 'v2' else mobile_base_body_xyz) if mobile_base else xyz}"
+        rpy="${('0 0 0' if body_type == 'v2' else mobile_base_body_rpy) if mobile_base else rpy}"
         inertials="${body_inertials}"
         kinematics="${body_kinematics}"
@@ -128,5 +141,7 @@
             gazebo="${gazebo}"
             hand="${hand}"
-            ee_type="${ee_type}"/>
+            ee_type="${ee_type}"
+            body_type="${body_type}"
+            no_prefix="${no_prefix}"/>
         </xacro:if>
         <xacro:if value="$(eval hand and ee_type == 'openarm_hand')">
@@ -196,9 +211,4 @@
                 rpy="$(arg rpy_ee)"
             />
-            <!-- The old ad-hoc 180-flip link that used to sit between
-                 openarm_right_link7 and the right connector is gone: it's
-                 now folded into connector_rpy_right's own mirror default
-                 (see amazing_hand_arguments.xacro), so right's connector
-                 attaches directly to link7 just like left's does. -->
             <xacro:amazing_hand_connector side="right" parent="openarm_right_link7"
                 xyz="$(arg connector_xyz_right)" rpy="$(arg connector_rpy_right)" />

File: Open_arm_a1_ws/src/openarm_description/urdf/robot/v10.urdf.xacro (robot description, xacro)
@@ -23,7 +23,7 @@
   <xacro:arg name="fake_sensor_commands" default="false" />
   <xacro:arg name="bimanual" default="false" />
-  <xacro:arg name="right_arm_base_xyz" default="-0.0964262 0.1302 0.836" />
+  <xacro:arg name="right_arm_base_xyz" default="-0.03 0.118 0.21" />
   <xacro:arg name="right_arm_base_rpy" default="1.5708 0 3.14159" />
-  <xacro:arg name="left_arm_base_xyz" default="-0.0964262 -0.1302 0.836" />
+  <xacro:arg name="left_arm_base_xyz" default="-0.03 -0.112 0.21" />
   <xacro:arg name="left_arm_base_rpy" default="-1.5708 0 3.14159" />
   <xacro:arg name="can_fd" default="true" />

File: Open_arm_a1_ws/src/openarm_description/urdf/ros2_control/openarm.bimanual.ros2_control.xacro (robot description, xacro)
@@ -14,5 +14,8 @@
              right_arm_prefix:=^|right_
              gazebo:=^|false
-             can_fd:=^|true">
+             can_fd:=^|true
+             body_type:=^|v1
+             no_prefix:=^|false">
+    <xacro:property name="body_joint_prefix" value="${'' if no_prefix else 'openarm_body_'}" />
     <xacro:macro name="configure_arm_joint" params="joint_name initial_position">
       <joint name="${joint_name}">
@@ -226,4 +229,27 @@
         <joint name="openarm_base_br_wheel_joint"><state_interface name="position"><param name="initial_value">0.0</param></state_interface></joint>
     </ros2_control>
+    <!-- body v2's articulated neck + head; no-op for v1 (rigid body has no such joints) -->
+    <xacro:if value="${body_type == 'v2'}">
+      <ros2_control name="openarm_head_hardware_interface" type="system">
+        <hardware>
+          <xacro:if value="${use_fake_hardware}">
+            <plugin>mock_components/GenericSystem</plugin>
+            <param name="fake_sensor_commands">${fake_sensor_commands}</param>
+            <param name="state_following_offset">0.0</param>
+          </xacro:if>
+          <xacro:unless value="${use_fake_hardware}">
+            <xacro:if value="${gazebo}">
+              <plugin>gz_ros2_control/GazeboSimSystem</plugin>
+            </xacro:if>
+            <xacro:unless value="${gazebo}">
+              <!-- Real robot driver if applicable -->
+              <plugin>mock_components/GenericSystem</plugin>
+            </xacro:unless>
+          </xacro:unless>
+        </hardware>
+        <xacro:configure_arm_joint joint_name="${body_joint_prefix}neck_joint" initial_position="0.0"/>
+        <xacro:configure_arm_joint joint_name="${body_joint_prefix}head_joint" initial_position="0.0"/>
+      </ros2_control>
+    </xacro:if>
   </xacro:macro>
   <gazebo>
