Commit message: refactor: update BehaviorTree.ROS2 and topic_based_ros2_control implementations and testing configurations

File: Open_arm_a1_ws/src/openarm_description/urdf/ros2_control/openarm.bimanual.ros2_control.xacro (robot description, xacro)
@@ -45,53 +45,28 @@
             </xacro:if>
             <xacro:unless value="${use_fake_hardware}">
-              <plugin>openarm_hardware/OpenArm_v10HW</plugin>
-              <param name="can_interface">${left_can_interface}</param>
-              <param name="arm_prefix">${left_arm_prefix}</param>
-              <param name="hand">${hand}</param>
-              <param name="can_fd">${can_fd}</param>
-              <param name="kp1">${control_gains['joint1']['kp']}</param>
-              <param name="kp2">${control_gains['joint2']['kp']}</param>
-              <param name="kp3">${control_gains['joint3']['kp']}</param>
-              <param name="kp4">${control_gains['joint4']['kp']}</param>
-              <param name="kp5">${control_gains['joint5']['kp']}</param>
-              <param name="kp6">${control_gains['joint6']['kp']}</param>
-              <param name="kp7">${control_gains['joint7']['kp']}</param>
-              <param name="kd1">${control_gains['joint1']['kd']}</param>
-              <param name="kd2">${control_gains['joint2']['kd']}</param>
-              <param name="kd3">${control_gains['joint3']['kd']}</param>
-              <param name="kd4">${control_gains['joint4']['kd']}</param>
-              <param name="kd5">${control_gains['joint5']['kd']}</param>
-              <param name="kd6">${control_gains['joint6']['kd']}</param>
-              <param name="kd7">${control_gains['joint7']['kd']}</param>
-            </xacro:unless>
-          <xacro:if value="${use_fake_hardware}">
-            <plugin>mock_components/GenericSystem</plugin>
-            <param name="fake_sensor_commands">${fake_sensor_commands}</param>
-            <param name="state_following_offset">0.0</param>
-          </xacro:if>
-          <xacro:unless value="${use_fake_hardware}">
-            <xacro:if value="${gazebo}">
-              <plugin>gz_ros2_control/GazeboSimSystem</plugin>
-            </xacro:if>
-            <xacro:unless value="${gazebo}">
-              <plugin>openarm_hardware/OpenArm_v10HW</plugin>
-              <param name="can_interface">${left_can_interface}</param>
-              <param name="arm_prefix">${left_arm_prefix}</param>
-              <param name="hand">${hand}</param>
-              <param name="can_fd">${can_fd}</param>
-              <param name="kp1">${control_gains['joint1']['kp']}</param>
-              <param name="kp2">${control_gains['joint2']['kp']}</param>
-              <param name="kp3">${control_gains['joint3']['kp']}</param>
-              <param name="kp4">${control_gains['joint4']['kp']}</param>
-              <param name="kp5">${control_gains['joint5']['kp']}</param>
-              <param name="kp6">${control_gains['joint6']['kp']}</param>
-              <param name="kp7">${control_gains['joint7']['kp']}</param>
-              <param name="kd1">${control_gains['joint1']['kd']}</param>
-              <param name="kd2">${control_gains['joint2']['kd']}</param>
-              <param name="kd3">${control_gains['joint3']['kd']}</param>
-              <param name="kd4">${control_gains['joint4']['kd']}</param>
-              <param name="kd5">${control_gains['joint5']['kd']}</param>
-              <param name="kd6">${control_gains['joint6']['kd']}</param>
-              <param name="kd7">${control_gains['joint7']['kd']}</param>
+              <xacro:if value="${gazebo}">
+                <plugin>gz_ros2_control/GazeboSimSystem</plugin>
+              </xacro:if>
+              <xacro:unless value="${gazebo}">
+                <plugin>openarm_hardware/OpenArm_v10HW</plugin>
+                <param name="can_interface">${left_can_interface}</param>
+                <param name="arm_prefix">${left_arm_prefix}</param>
+                <param name="hand">${hand}</param>
+                <param name="can_fd">${can_fd}</param>
+                <param name="kp1">${control_gains['joint1']['kp']}</param>
+                <param name="kp2">${control_gains['joint2']['kp']}</param>
+                <param name="kp3">${control_gains['joint3']['kp']}</param>
+                <param name="kp4">${control_gains['joint4']['kp']}</param>
+                <param name="kp5">${control_gains['joint5']['kp']}</param>
+                <param name="kp6">${control_gains['joint6']['kp']}</param>
+                <param name="kp7">${control_gains['joint7']['kp']}</param>
+                <param name="kd1">${control_gains['joint1']['kd']}</param>
+                <param name="kd2">${control_gains['joint2']['kd']}</param>
+                <param name="kd3">${control_gains['joint3']['kd']}</param>
+                <param name="kd4">${control_gains['joint4']['kd']}</param>
+                <param name="kd5">${control_gains['joint5']['kd']}</param>
+                <param name="kd6">${control_gains['joint6']['kd']}</param>
+                <param name="kd7">${control_gains['joint7']['kd']}</param>
+              </xacro:unless>
             </xacro:unless>
           </xacro:unless>
@@ -104,25 +79,35 @@
       <xacro:configure_arm_joint joint_name="openarm_${left_arm_prefix}joint6" initial_position="0.0"/>
       <xacro:configure_arm_joint joint_name="openarm_${left_arm_prefix}joint7" initial_position="0.0"/>
-      <xacro:if value="${hand}">
-        <xacro:configure_joint joint_name="openarm_${left_arm_prefix}finger_joint1" initial_position="0.0" />
-        <xacro:if value="${use_isaac_sim}">
-          <joint name="openarm_${left_arm_prefix}finger_joint2">
-            <param name="mimic">openarm_${left_arm_prefix}finger_joint1</param>
-            <param name="multiplier">1.0</param>
-            <state_interface name="position">
-              <param name="initial_value">0.0</param>
-            </state_interface>
-            <state_interface name="velocity">
-              <param name="initial_value">0.0</param>
-            </state_interface>
-            <state_interface name="effort">
-              <param name="initial_value">0.0</param>
-            </state_interface>
-          </joint>
-        </xacro:if>
+    </ros2_control>
+    <!-- LEFT GRIPPER -->
+    <xacro:if value="${hand}">
+      <ros2_control name="openarm_left_gripper_hardware_interface" type="system">
+        <hardware>
+          <xacro:if value="${use_isaac_sim}">
+            <plugin>topic_based_ros2_control/TopicBasedSystem</plugin>
+            <param name="joint_commands_topic">/isaac_left_gripper/joint_commands</param>
+            <param name="joint_states_topic">/isaac_left_gripper/joint_states</param>
+          </xacro:if>
+          <xacro:unless value="${use_isaac_sim}">
+            <xacro:if value="${use_fake_hardware}">
+              <plugin>mock_components/GenericSystem</plugin>
+              <param name="fake_sensor_commands">${fake_sensor_commands}</param>
+              <param name="state_following_offset">0.0</param>
+            </xacro:if>
+            <xacro:unless value="${use_fake_hardware}">
+              <xacro:if value="${gazebo}">
+                <plugin>gz_ros2_control/GazeboSimSystem</plugin>
+              </xacro:if>
+              <xacro:unless value="${gazebo}">
+                <!-- Real robot driver if applicable -->
+                <plugin>mock_components/GenericSystem</plugin>
+              </xacro:unless>
+            </xacro:unless>
+          </xacro:unless>
+        </hardware>
         <xacro:configure_arm_joint joint_name="openarm_${left_arm_prefix}finger_joint1" initial_position="0.0" />
         <xacro:configure_arm_joint joint_name="openarm_${left_arm_prefix}finger_joint2" initial_position="0.0" />
-      </xacro:if>
-    </ros2_control>
+      </ros2_control>
+    </xacro:if>
     <ros2_control name="openarm_right_hardware_interface" type="system">
         <hardware>
@@ -140,53 +125,28 @@
             </xacro:if>
             <xacro:unless value="${use_fake_hardware}">
-              <plugin>openarm_hardware/OpenArm_v10HW</plugin>
-              <param name="can_interface">${right_can_interface}</param>
-              <param name="arm_prefix">${right_arm_prefix}</param>
-              <param name="hand">${hand}</param>
-              <param name="can_fd">${can_fd}</param>
-              <param name="kp1">${control_gains['joint1']['kp']}</param>
-              <param name="kp2">${control_gains['joint2']['kp']}</param>
-              <param name="kp3">${control_gains['joint3']['kp']}</param>
-              <param name="kp4">${control_gains['joint4']['kp']}</param>
-              <param name="kp5">${control_gains['joint5']['kp']}</param>
-              <param name="kp6">${control_gains['joint6']['kp']}</param>
-              <param name="kp7">${control_gains['joint7']['kp']}</param>
-              <param name="kd1">${control_gains['joint1']['kd']}</param>
-              <param name="kd2">${control_gains['joint2']['kd']}</param>
-              <param name="kd3">${control_gains['joint3']['kd']}</param>
-              <param name="kd4">${control_gains['joint4']['kd']}</param>
-              <param name="kd5">${control_gains['joint5']['kd']}</param>
-              <param name="kd6">${control_gains['joint6']['kd']}</param>
-              <param name="kd7">${control_gains['joint7']['kd']}</param>
-            </xacro:unless>
-          <xacro:if value="${use_fake_hardware}">
-            <plugin>mock_components/GenericSystem</plugin>
-            <param name="fake_sensor_commands">${fake_sensor_commands}</param>
-            <param name="state_following_offset">0.0</param>
-          </xacro:if>
-          <xacro:unless value="${use_fake_hardware}">
-            <xacro:if value="${gazebo}">
-              <plugin>gz_ros2_control/GazeboSimSystem</plugin>
-            </xacro:if>
-            <xacro:unless value="${gazebo}">
-              <plugin>openarm_hardware/OpenArm_v10HW</plugin>
-              <param name="can_interface">${right_can_interface}</param>
-              <param name="arm_prefix">${right_arm_prefix}</param>
-              <param name="hand">${hand}</param>
-              <param name="can_fd">${can_fd}</param>
-              <param name="kp1">${control_gains['joint1']['kp']}</param>
-              <param name="kp2">${control_gains['joint2']['kp']}</param>
-              <param name="kp3">${control_gains['joint3']['kp']}</param>
-              <param name="kp4">${control_gains['joint4']['kp']}</param>
-              <param name="kp5">${control_gains['joint5']['kp']}</param>
-              <param name="kp6">${control_gains['joint6']['kp']}</param>
-              <param name="kp7">${control_gains['joint7']['kp']}</param>
-              <param name="kd1">${control_gains['joint1']['kd']}</param>
-              <param name="kd2">${control_gains['joint2']['kd']}</param>
-              <param name="kd3">${control_gains['joint3']['kd']}</param>
-              <param name="kd4">${control_gains['joint4']['kd']}</param>
-              <param name="kd5">${control_gains['joint5']['kd']}</param>
-              <param name="kd6">${control_gains['joint6']['kd']}</param>
-              <param name="kd7">${control_gains['joint7']['kd']}</param>
+              <xacro:if value="${gazebo}">
+                <plugin>gz_ros2_control/GazeboSimSystem</plugin>
+              </xacro:if>
+              <xacro:unless value="${gazebo}">
+                <plugin>openarm_hardware/OpenArm_v10HW</plugin>
+                <param name="can_interface">${right_can_interface}</param>
+                <param name="arm_prefix">${right_arm_prefix}</param>
+                <param name="hand">${hand}</param>
+                <param name="can_fd">${can_fd}</param>
+                <param name="kp1">${control_gains['joint1']['kp']}</param>
+                <param name="kp2">${control_gains['joint2']['kp']}</param>
+                <param name="kp3">${control_gains['joint3']['kp']}</param>
+                <param name="kp4">${control_gains['joint4']['kp']}</param>
+                <param name="kp5">${control_gains['joint5']['kp']}</param>
+                <param name="kp6">${control_gains['joint6']['kp']}</param>
+                <param name="kp7">${control_gains['joint7']['kp']}</param>
+                <param name="kd1">${control_gains['joint1']['kd']}</param>
+                <param name="kd2">${control_gains['joint2']['kd']}</param>
+                <param name="kd3">${control_gains['joint3']['kd']}</param>
+                <param name="kd4">${control_gains['joint4']['kd']}</param>
+                <param name="kd5">${control_gains['joint5']['kd']}</param>
+                <param name="kd6">${control_gains['joint6']['kd']}</param>
+                <param name="kd7">${control_gains['joint7']['kd']}</param>
+              </xacro:unless>
             </xacro:unless>
           </xacro:unless>
@@ -199,25 +159,35 @@
       <xacro:configure_arm_joint joint_name="openarm_${right_arm_prefix}joint6" initial_position="0.0"/>
       <xacro:configure_arm_joint joint_name="openarm_${right_arm_prefix}joint7" initial_position="0.0"/>
-      <xacro:if value="${hand}">
-        <xacro:configure_joint joint_name="openarm_${right_arm_prefix}finger_joint1" initial_position="0.0" />
-        <xacro:if value="${use_isaac_sim}">
-          <joint name="openarm_${right_arm_prefix}finger_joint2">
-            <param name="mimic">openarm_${right_arm_prefix}finger_joint1</param>
-            <param name="multiplier">1.0</param>
-            <state_interface name="position">
-              <param name="initial_value">0.0</param>
-            </state_interface>
-            <state_interface name="velocity">
-              <param name="initial_value">0.0</param>
-            </state_interface>
-            <state_interface name="effort">
-              <param name="initial_value">0.0</param>
-            </state_interface>
-          </joint>
-        </xacro:if>
+    </ros2_control>
+    <!-- RIGHT GRIPPER -->
+    <xacro:if value="${hand}">
+      <ros2_control name="openarm_right_gripper_hardware_interface" type="system">
+        <hardware>
+          <xacro:if value="${use_isaac_sim}">
+            <plugin>topic_based_ros2_control/TopicBasedSystem</plugin>
+            <param name="joint_commands_topic">/isaac_right_gripper/joint_commands</param>
+            <param name="joint_states_topic">/isaac_right_gripper/joint_states</param>
+          </xacro:if>
+          <xacro:unless value="${use_isaac_sim}">
+            <xacro:if value="${use_fake_hardware}">
+              <plugin>mock_components/GenericSystem</plugin>
+              <param name="fake_sensor_commands">${fake_sensor_commands}</param>
+              <param name="state_following_offset">0.0</param>
+            </xacro:if>
+            <xacro:unless value="${use_fake_hardware}">
+              <xacro:if value="${gazebo}">
+                <plugin>gz_ros2_control/GazeboSimSystem</plugin>
+              </xacro:if>
+              <xacro:unless value="${gazebo}">
+                <!-- Real robot driver if applicable -->
+                <plugin>mock_components/GenericSystem</plugin>
+              </xacro:unless>
+            </xacro:unless>
+          </xacro:unless>
+        </hardware>
         <xacro:configure_arm_joint joint_name="openarm_${right_arm_prefix}finger_joint1" initial_position="0.0" />
         <xacro:configure_arm_joint joint_name="openarm_${right_arm_prefix}finger_joint2" initial_position="0.0" />
-      </xacro:if>
-    </ros2_control>
+      </ros2_control>
+    </xacro:if>
     <ros2_control name="openarm_base_hardware_interface" type="system">
         <hardware>
