Commit message: feat: add amazing hand connector and tuning parameters for improved end-effector integration

File: Open_arm_a1_ws/src/openarm_description/urdf/ee/amazing_hand_arguments.xacro (robot description, xacro)
@@ -3,10 +3,42 @@
   <!-- Where is the end-effector connected to, if different from the robot flange?  -->
   <xacro:arg name="special_connection" default="" />
-  <!-- Position offset between the arm's wrist flange and the hand's root link.
-       Not yet calibrated against real hardware: the standalone amazing_hand
-       display/control launches place root at the world origin directly, so
-       this mount transform is an untested placeholder. Expect to tune it. -->
-  <xacro:arg name="xyz_ee" default="0 0 0" />
-  <xacro:arg name="rpy_ee" default="0 0 0" />
+  <!-- Hand mount: position/rotation of the hand's root link relative to the
+       connector (left side; right has its own override below). Empirically
+       tuned in RViz against real hardware. -->
+  <xacro:arg name="xyz_ee" default="0.0358 -0.0148 0.1" />
+  <xacro:arg name="rpy_ee" default="0 0 -1.047" />
+  <!-- Right-hand-only overrides. Left is untouched by these. Also tuned
+       empirically; not a pure mirror of xyz_ee/rpy_ee (a geometric mirror
+       about the body's Y=0 plane gets close but doesn't match real hardware
+       exactly, position and rotation both needed further hand adjustment). -->
+  <xacro:arg name="xyz_ee_right" default="0.0358 0.0148 0.1" />
+  <xacro:arg name="rpy_ee_right" default="0 0 4.1887" />
+  <!-- Physical connector plate between the arm's wrist flange and the hand's
+       root link (meshes/ee/amazing_hand/{visual,collision}/connector.STL).
+       Position/rotation of the connector's own origin relative to link7;
+       the hand mount above is then relative to THIS link, not to link7
+       directly. Shared fallback for both sides; connector_*_left/right
+       below override per side. Empirically tuned; the shared fallback here
+       is what left actually uses (connector_xyz_left/connector_rpy_left
+       just default to these). -->
+  <xacro:arg name="connector_xyz" default="0 0 0.0055" />
+  <xacro:arg name="connector_rpy" default="0 0 1.047" />
+  <!-- Per-side connector overrides, on top of connector_xyz/connector_rpy
+       above. Each only touches its own side. Rotating a connector alone
+       also rotates that side's hand (parent-child propagation); compensate
+       via rpy_ee (left) / rpy_ee_right (right) if the hand needs to hold
+       its orientation. Right's default is the Y=0-plane mirror of left's
+       (Z: 1.047 -> -1.047); there is no separate "flip" joint in the
+       URDF, right's connector attaches directly to openarm_right_link7,
+       same as left's does to openarm_left_link7. -->
+  <xacro:arg name="connector_xyz_left" default="$(arg connector_xyz)" />
+  <xacro:arg name="connector_rpy_left" default="$(arg connector_rpy)" />
+  <xacro:arg name="connector_xyz_right" default="0 0 0.0055" />
+  <xacro:arg name="connector_rpy_right" default="0 0 -1.047" />
+  <!-- connector.STL bounding box is ~49x49x11 in file units; that reads as
+       millimeters against the rest of this URDF (meters), hence 0.001 scale.
+       If it renders house-sized or invisible-tiny in RViz, this guess is
+       backwards, try "1 1 1" instead. -->
+  <xacro:arg name="connector_scale" default="0.001 0.001 0.001" />
   <!-- Position/rotation offset between ee frame and tcp frame, unused by
        amazing_hand today; kept for interface parity with openarm_hand. -->

File: Open_arm_a1_ws/src/openarm_description/urdf/robot/openarm_robot.xacro (robot description, xacro)
@@ -159,15 +159,53 @@
           </xacro:if>
         <xacro:if value="$(eval hand and ee_type == 'amazing_hand')">
+            <!-- Physical connector plate between the arm flange and the hand
+                 root (see amazing_hand_arguments.xacro for connector_xyz/
+                 connector_rpy/connector_xyz_left/connector_rpy_left/
+                 connector_scale). One macro, instantiated once per side since
+                 each needs its own link/joint names and can take its own
+                 mount xyz/rpy. -->
+            <xacro:macro name="amazing_hand_connector" params="side parent xyz rpy">
+                <link name="openarm_${side}_ahand_connector">
+                    <visual>
+                        <origin xyz="0 0 -0.035" rpy="0 0 0" />
+                        <geometry>
+                            <mesh filename="package://openarm_description/meshes/ee/amazing_hand/visual/connector.STL"
+                                  scale="$(arg connector_scale)" />
+                        </geometry>
+                    </visual>
+                    <collision>
+                        <origin xyz="0 0 0" rpy="0 0 0" />
+                        <geometry>
+                            <mesh filename="package://openarm_description/meshes/ee/amazing_hand/collision/connector.STL"
+                                  scale="$(arg connector_scale)" />
+                        </geometry>
+                    </collision>
+                </link>
+                <joint name="openarm_${side}_ahand_connector_joint" type="fixed">
+                    <origin xyz="${xyz}" rpy="${rpy}" />
+                    <parent link="${parent}" />
+                    <child link="openarm_${side}_ahand_connector" />
+                </joint>
+            </xacro:macro>
+            <xacro:amazing_hand_connector side="left" parent="openarm_left_link7"
+                xyz="$(arg connector_xyz_left)" rpy="$(arg connector_rpy_left)" />
             <xacro:amazing_hand_left
-                connected_to="openarm_left_link7"
+                connected_to="openarm_left_ahand_connector"
                 prefix="openarm_left_ahand_"
                 xyz="$(arg xyz_ee)"
                 rpy="$(arg rpy_ee)"
             />
+            <!-- The old ad-hoc 180-flip link that used to sit between
+                 openarm_right_link7 and the right connector is gone: it's
+                 now folded into connector_rpy_right's own mirror default
+                 (see amazing_hand_arguments.xacro), so right's connector
+                 attaches directly to link7 just like left's does. -->
+            <xacro:amazing_hand_connector side="right" parent="openarm_right_link7"
+                xyz="$(arg connector_xyz_right)" rpy="$(arg connector_rpy_right)" />
             <xacro:amazing_hand_right
-                connected_to="openarm_right_link7"
+                connected_to="openarm_right_ahand_connector"
                 prefix="openarm_right_ahand_"
-                xyz="$(arg xyz_ee)"
-                rpy="$(arg rpy_ee)"
+                xyz="$(arg xyz_ee_right)"
+                rpy="$(arg rpy_ee_right)"
             />
             <!-- left_arm/right_arm MoveIt groups (defined once, shared across

Commit message: home position at -10 and 10

File: Open_arm_a1_ws/src/openarm_description/urdf/ee/amazing_hand_arguments.xacro (robot description, xacro)
@@ -45,4 +45,18 @@
   <xacro:arg name="tcp_xyz" default="0 0 0" />
   <xacro:arg name="tcp_rpy" default="0 0 0" />
+  <!-- Hand-rotate axis ("motor 8" - the same physical CAN motor that drove
+       openarm_hand's finger_joint1 gripper actuator; on amazing_hand rigs it
+       instead spins the whole hand via the connector, through a mechanism
+       external to this URDF). Axis is in the connector_joint's own frame
+       (post connector_rpy rotation). VERIFY against the real mechanism
+       before running on hardware - wrong axis/limits will drive the motor
+       into a mechanical hard stop. -->
+  <xacro:arg name="hand_rotate_axis" default="0 0 1" />
+  <!-- Same as arm joint7 (also a DM4310) - a placeholder, not a measured
+       value for this mechanism. -->
+  <xacro:arg name="hand_rotate_lower" default="-1.570796" />
+  <xacro:arg name="hand_rotate_upper" default="1.570796" />
+  <xacro:arg name="hand_rotate_effort" default="12.0" />
+  <xacro:arg name="hand_rotate_velocity" default="2.0" />
   <!-- Name of the description package -->
   <xacro:arg name="description_pkg" default="openarm_description" />

File: Open_arm_a1_ws/src/openarm_description/urdf/robot/openarm_robot.xacro (robot description, xacro)
@@ -150,4 +150,5 @@
             body_type="${body_type}"
             no_prefix="${no_prefix}"
+            hand_rotate_ratio="$(arg hand_rotate_ratio)"
             shutdown_disable_retries="${shutdown_disable_retries}"
             shutdown_retry_delay_ms="${shutdown_retry_delay_ms}"
@@ -238,8 +239,22 @@
                     </inertial>
                 </link>
-                <joint name="openarm_${side}_ahand_connector_joint" type="fixed">
+                <!-- "Motor 8": the same real CAN motor (DM4310, id 0x08) that
+                     drives openarm_hand's finger_joint1 gripper actuator -
+                     hand_ is xacro-arg "hand" (default true) independent of
+                     ee_type, so OpenArm_v10HW already exports a
+                     command/state interface named openarm_${side}_finger_joint1
+                     regardless of which end-effector is attached (see
+                     generate_joint_names() in hardware_interface.cpp). Naming
+                     this joint the same lets that pre-existing interface
+                     attach here instead of floating unclaimed. Axis/limits
+                     are placeholders - verify against the real mechanism
+                     before running on hardware (see amazing_hand_arguments.xacro). -->
+                <joint name="openarm_${side}_finger_joint1" type="revolute">
                     <origin xyz="${xyz}" rpy="${rpy}" />
                     <parent link="${parent}" />
                     <child link="openarm_${side}_ahand_connector" />
+                    <axis xyz="$(arg hand_rotate_axis)" />
+                    <limit lower="$(arg hand_rotate_lower)" upper="$(arg hand_rotate_upper)"
+                           effort="$(arg hand_rotate_effort)" velocity="$(arg hand_rotate_velocity)" />
                 </joint>
             </xacro:macro>
@@ -313,4 +328,5 @@
             fake_sensor_commands="${fake_sensor_commands}"
             hand="${hand}"
+            hand_rotate_ratio="$(arg hand_rotate_ratio)"
             ee_type="${ee_type}"
             bimanual="false"

File: Open_arm_a1_ws/src/openarm_description/urdf/robot/v10.urdf.xacro (robot description, xacro)
@@ -7,4 +7,5 @@
   <xacro:arg name="no_prefix" default="false"/>
   <xacro:arg name="hand" default="true" />
+  <xacro:arg name="hand_rotate_ratio" default="1.0" />
   <xacro:if value="$(eval ee_type == 'none')">
     <xacro:property name="hand" value="false"/>

File: Open_arm_a1_ws/src/openarm_description/urdf/ros2_control/openarm.bimanual.ros2_control.xacro (robot description, xacro)
@@ -10,4 +10,5 @@
              fake_sensor_commands:=^|false
              hand:=^|false
+             hand_rotate_ratio:=^|1.0
              ee_type:=^|openarm_hand
              left_arm_prefix:=^|left_
@@ -57,4 +58,5 @@
               <param name="arm_prefix">${left_arm_prefix}</param>
               <param name="hand">${hand}</param>
+              <param name="hand_rotate_ratio">${hand_rotate_ratio}</param>
               <param name="can_fd">${can_fd}</param>
               <param name="control_mode">${control_mode}</param>
@@ -82,5 +84,12 @@
         </hardware>
       <xacro:configure_arm_joint joint_name="openarm_${left_arm_prefix}joint1" initial_position="0.0"/>
-      <xacro:configure_arm_joint joint_name="openarm_${left_arm_prefix}joint2" initial_position="0.0"/>
+      <!-- Cosmetic sim-only spawn pose matching the "motor8_safe" SRDF
+           group_state (openarm_bimanual.srdf) - RViz/fake hardware starts
+           already angled out instead of straight, no separate "move to
+           safe pose" step needed just to look at it. Real hardware
+           (OpenArm_v10HW) ignores this entirely and reports actual encoder
+           position instead - use motor8_safe (a real commanded trajectory)
+           there, not this. -->
+      <xacro:configure_arm_joint joint_name="openarm_${left_arm_prefix}joint2" initial_position="-0.174533"/>
       <xacro:configure_arm_joint joint_name="openarm_${left_arm_prefix}joint3" initial_position="0.0"/>
       <xacro:configure_arm_joint joint_name="openarm_${left_arm_prefix}joint4" initial_position="0.0"/>
@@ -118,4 +127,31 @@
       </ros2_control>
     </xacro:if>
+    <!-- LEFT "MOTOR 8" (amazing_hand's connector rotation - openarm_hand's
+         finger_joint2 has no equivalent here, the connector is a single
+         joint). Same fake/gazebo-only reasoning as the gripper block above:
+         openarm_left_hardware_interface's OpenArm_v10HW owns this joint for
+         real; on the fake/gazebo path that plugin is swapped out for
+         mock_components/GenericSystem, which (unlike OpenArm_v10HW) only
+         exports interfaces for joints actually declared in ITS OWN
+         <ros2_control> block - and openarm_left_hardware_interface only
+         declares joint1..7 there, so finger_joint1 needs its own mock
+         component or it silently has no interfaces on this path at all
+         (JointTrajectoryController goals get rejected with no reason
+         logged). -->
+    <xacro:if value="${hand and ee_type == 'amazing_hand' and (use_fake_hardware or gazebo)}">
+      <ros2_control name="openarm_left_hand_rotate_hardware_interface" type="system">
+        <hardware>
+          <xacro:if value="${use_fake_hardware}">
+            <plugin>mock_components/GenericSystem</plugin>
+            <param name="fake_sensor_commands">${fake_sensor_commands}</param>
+            <param name="state_following_offset">0.0</param>
+          </xacro:if>
+          <xacro:unless value="${use_fake_hardware}">
+            <plugin>gz_ros2_control/GazeboSimSystem</plugin>
+          </xacro:unless>
+        </hardware>
+        <xacro:configure_arm_joint joint_name="openarm_${left_arm_prefix}finger_joint1" initial_position="0.0" />
+      </ros2_control>
+    </xacro:if>
     <ros2_control name="openarm_right_hardware_interface" type="system">
         <hardware>
@@ -135,4 +171,5 @@
               <param name="arm_prefix">${right_arm_prefix}</param>
               <param name="hand">${hand}</param>
+              <param name="hand_rotate_ratio">${hand_rotate_ratio}</param>
               <param name="can_fd">${can_fd}</param>
               <param name="control_mode">${control_mode}</param>
@@ -160,5 +197,7 @@
         </hardware>
       <xacro:configure_arm_joint joint_name="openarm_${right_arm_prefix}joint1" initial_position="0.0"/>
-      <xacro:configure_arm_joint joint_name="openarm_${right_arm_prefix}joint2" initial_position="0.0"/>
+      <!-- See left_hardware_interface's joint2 comment above - mirrors
+           motor8_safe's right_arm sign (+ instead of -). -->
+      <xacro:configure_arm_joint joint_name="openarm_${right_arm_prefix}joint2" initial_position="0.174533"/>
       <xacro:configure_arm_joint joint_name="openarm_${right_arm_prefix}joint3" initial_position="0.0"/>
       <xacro:configure_arm_joint joint_name="openarm_${right_arm_prefix}joint4" initial_position="0.0"/>
@@ -194,4 +233,21 @@
         </xacro:if>
         <xacro:configure_arm_joint joint_name="openarm_${right_arm_prefix}finger_joint2" initial_position="0.0" />
+      </ros2_control>
+    </xacro:if>
+    <!-- RIGHT "MOTOR 8" - see openarm_left_hand_rotate_hardware_interface's
+         comment above. -->
+    <xacro:if value="${hand and ee_type == 'amazing_hand' and (use_fake_hardware or gazebo)}">
+      <ros2_control name="openarm_right_hand_rotate_hardware_interface" type="system">
+        <hardware>
+          <xacro:if value="${use_fake_hardware}">
+            <plugin>mock_components/GenericSystem</plugin>
+            <param name="fake_sensor_commands">${fake_sensor_commands}</param>
+            <param name="state_following_offset">0.0</param>
+          </xacro:if>
+          <xacro:unless value="${use_fake_hardware}">
+            <plugin>gz_ros2_control/GazeboSimSystem</plugin>
+          </xacro:unless>
+        </hardware>
+        <xacro:configure_arm_joint joint_name="openarm_${right_arm_prefix}finger_joint1" initial_position="0.0" />
       </ros2_control>
     </xacro:if>

File: Open_arm_a1_ws/src/openarm_description/urdf/ros2_control/openarm.ros2_control.xacro (robot description, xacro)
@@ -8,4 +8,5 @@
              fake_sensor_commands:=^|false
              hand:=^|false
+             hand_rotate_ratio:=^|1.0
              ee_type:=^|openarm_hand
              gazebo_effort:=^|false
@@ -27,4 +28,5 @@
             <param name="arm_prefix">${arm_prefix}</param>
             <param name="hand">${hand}</param>
+            <param name="hand_rotate_ratio">${hand_rotate_ratio}</param>
             <param name="can_fd">${can_fd}</param>
             <param name="kp1">${control_gains['joint1']['kp']}</param>
